File: PCB/Main Board/PGS_Main_Board.kicad_sch (KiCad schematic)
At the start: 132 parts, among them J1 SM02B-SURS-TF_LF__SN_, J2 SM02B-SURS-TF_LF__SN_, J3 Molex 505110-0892, J5 Molex 505110-0892, J6 Molex 505110-0492, J7 Molex 505110-0492, J8 Conn_01x04_Pin, J9 Molex 505110-1792, Q1 MMBT2222A, Q2 MMBT2222A, SW1 TS-1187A-C-A-B, SW10 SW_Push, SW11 SW_Push, SW12 SW_Push, SW13 SW_Push, SW14 EVQ-P0E07K, SW15 1TS026A-1000-0550, SW16 TS-1187A-C-A-B, SW2 TS-1187A-C-A-B, SW3 TS-1187A-C-A-B, SW4 TS-1187A-C-A-B, SW5 SW_Push, SW6 SW_Push, SW7 SW_Push, SW8 SW_Push, SW9 EVQ-P0E07K, U1 RP2040, U2 TPS630001RCR, U3 GD25Q80EEIGR, U4 ST_LSM6, U5 ST_LSM6, Y1 ABM8-272-T3

Commit message: PCB Routing
Parts:
- J1, J2: Package SMD,P=0.8mm,Surface Mount，Right Angle -> None
Connections:
- net ADC_ADDR_0: now also U1.38 (GPIO26_ADC0); no longer U1.31 (GPIO20)
- net ADC_ADDR_1: now also U1.39 (GPIO27_ADC1); no longer U1.32 (GPIO21)
- net D+: now also J9.15 (Pin_15); no longer J9.13 (Pin_13)
- net D-: now also J9.16 (Pin_16); no longer J9.14 (Pin_14)
- net I2C0_SCL: now also U1.28 (GPIO17); no longer U1.37 (GPIO25)
- net I2C0_SDA: now also U1.27 (GPIO16); no longer U1.36 (GPIO24)
- net VBUS_SYS: now also J9.13 (Pin_13), J9.14 (Pin_14); no longer J9.15 (Pin_15), J9.16 (Pin_16)
- net at D15.1 (A): now also SW12.2; no longer SW10.2
- net DI-: now reaches R4.2, U1.46 (USB_DM)
- net DI+: now reaches R3.2, U1.47 (USB_DP)
- net at SW14.2: now also D15.3 (A); no longer D16.2 (A)
- net at R21.1: no longer U1.27 (GPIO16)
- net at R22.1: no longer U1.28 (GPIO17)
- net at U1.30 (GPIO19): no longer R24.1
- net at SW8.2: now also D13.2 (A); no longer D14.1 (A)
- net at SW11.2: now also D16.1 (A); no longer D15.2 (A)
- net at SW13.2: now also D15.2 (A); no longer D16.1 (A)
- net at D13.3 (A): now also SW6.2; no longer SW7.2
- net at D14.2 (A): now also SW7.2; no longer SW9.2
- net at SW5.2: now also D14.1 (A); no longer D13.1 (A)
- new net: R24.1, U1.37 (GPIO25)
- new net: D16.2 (A), SW10.2
- new net: D13.1 (A), SW9.2
Other:
- moved on the sheet: C28, S1

Commit message: Routing update
Parts:
- removed C15, C17: 10uF, Capacitor_SMD:C_0805_2012Metric, symbol Device:C
- removed C16: 100nF, Capacitor_SMD:C_0201_0603Metric, symbol Device:C
- removed D7: CUS08F30,H3F, Diode_SMD:D_SOD-323_HandSoldering, symbol progcc_v3:CUS08F30
- removed L1: 1.3A 2.2uH ±20% 80mΩ, Inductor_SMD:L_1008_2520Metric, symbol Device:L
- removed R23: 100R, Resistor_SMD:R_0201_0603Metric, symbol Device:R
- removed TP1, TP2, TP3, TP4: TestPoint, TestPoint:TestPoint_Pad_2.0x2.0mm, symbol Connector:TestPoint
- removed TP5: TestPoint, TestPoint:TestPoint_Pad_D1.5mm, symbol Connector:TestPoint
- removed U2: TPS630001RCR, hhl:VREG_V62_16624-01YE, symbol hhl:TPS63000DRCR
- R11: LCSC C77623 -> C273268; Link https://www.lcsc.com/product-detail/Chip-Resistor-Surface-Mount_YAGEO-RC0201FR-07100RL_C77623.html -> https://www.lcsc.com/product-detail/Chip-Resistor-Surface-Mount_YAGEO-RC0201FR-0727RL_C273268.html; MPN RC0201FR-07100RL -> RC0201FR-0727RL
Connections:
- net LX is gone; now on net STICK_R_Y_OUT: S1.4 (S3)
- net LY is gone; now on net STICK_R_X_OUT: S1.2 (S1)
- net RX is gone; now on net STICK_L_X_OUT: S1.7 (S4)
- net RY is gone; now on net STICK_L_Y_OUT: S1.9 (S2)
- net +3V3: now also J9.13 (Pin_13), J9.14 (Pin_14)
- net A: now also D9.5 (K), R11.2; no longer D8.6 (K)
- net B: now also D9.6 (K); no longer D8.5 (K)
- net D: now also D8.5 (K); no longer D9.6 (K)
- net E: now also D8.6 (K); no longer D9.5 (K)
- net F: now also J3.7 (Pin_7), J7.1 (Pin_1), J7.4 (Pin_4), SW3.A, SW3.B, SW4.A, SW4.B; no longer J5.7 (Pin_7), J6.1 (Pin_1), J6.4 (Pin_4), SW1.A, SW1.B, SW2.A, SW2.B
- net G: now also J5.7 (Pin_7), J6.1 (Pin_1), J6.4 (Pin_4), SW1.A, SW1.B, SW2.A, SW2.B; no longer J3.7 (Pin_7), J7.1 (Pin_1), J7.4 (Pin_4), SW3.A, SW3.B, SW4.A, SW4.B
- net STICK_L_BTN_OUT: now also D9.1 (A); no longer D9.2 (A)
- net T_ZL_OUT: now also D8.2 (A); no longer D9.1 (A)
- net T_ZR_OUT: now also D11.2 (A); no longer D12.1 (A)
- net VBUS_SYS: no longer J9.13 (Pin_13), J9.14 (Pin_14), R11.1
- net at U1.13 (GPIO10): now also R11.1; no longer R15.1
- net at U1.14 (GPIO11): now also R22.1; no longer R16.1
- net at U1.15 (GPIO12): now also R21.1; no longer R17.1
- net at U1.16 (GPIO13): now also R20.1; no longer R18.1
- net at U1.18 (GPIO15): now also R18.1; no longer R20.1
- net at SW4.C, SW4.D: now also D12.1 (A); no longer D11.2 (A)
- net at SW2.C, SW2.D: now also D9.2 (A); no longer D8.2 (A)
Other:
- note removed: "3.3 Regulation"
- moved on the sheet: D11B, D12A, D8B, D9A, D9B, R19, R21, R22

Commit message: More Routing
Connections:
- net F: now also J5.7 (Pin_7), J6.1 (Pin_1), J6.4 (Pin_4), SW1.A, SW1.B, SW2.A, SW2.B; no longer J3.7 (Pin_7), J7.1 (Pin_1), J7.4 (Pin_4), SW3.A, SW3.B, SW4.A, SW4.B
- net G: now also J3.7 (Pin_7), J7.1 (Pin_1), J7.4 (Pin_4), SW3.A, SW3.B, SW4.A, SW4.B; no longer J5.7 (Pin_7), J6.1 (Pin_1), J6.4 (Pin_4), SW1.A, SW1.B, SW2.A, SW2.B
- net LRA_L: now also U1.31 (GPIO20); no longer U1.34 (GPIO22)
- net LRA_R: now also U1.32 (GPIO21); no longer U1.35 (GPIO23)
- net STICK_R_X_OUT: now also S1.4 (S3); no longer S1.2 (S1)
- net STICK_R_Y_OUT: now also S1.2 (S1); no longer S1.4 (S3)
- net at U1.29 (GPIO18): now also R16.1
- net at U1.30 (GPIO19): now also R15.1
- net at R17.1: now also U1.34 (GPIO22)
Other:
- moved on the sheet: R16, R17

Commit message: Routing/Labelling
Parts:
- removed C19: 100nF, Capacitor_SMD:C_0201_0603Metric, symbol Device:C
- C28: footprint Capacitor_SMD:C_0402_1005Metric -> Capacitor_SMD:C_0201_0603Metric
Connections:
- net A: now also D12.5 (K); no longer D11.6 (K)
- net B: now also D12.6 (K); no longer D11.5 (K)
- net D: now also D11.5 (K); no longer D12.6 (K)
- net E: now also D11.6 (K); no longer D12.5 (K)
