File: PCB/USBW Board/PGS_USBW_Board.kicad_pcb (KiCad board)
At the start: 4 copper layers, 49.1 x 32.6 mm, 44 parts, among them J1 Molex 505110-1792, J2 USB4056-03-A, J4 Adafruit 1769, P1 RPI-RM2, Q1 BSS138DW, Q2 BSS138DW, U1 USBLC6-2P6, U2 USBLC6-2P6, U3 USBLC6-2P6, U4 TPS63001DRCR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

Commit message: Final Routing 3D Export
- Export 3D STEP models
Other:
- board text added: "ProGCC 4 USB+W Module"
- board text removed: "PROGCC 4 COMMS&POWER+ PCB"
