File: PCB/Projects/Trigger Board/PGS_Trigger_Board.kicad_pcb (KiCad board)
At the start: 2 copper layers, 19 x 22 mm, 3 parts, among them J1 Molex 505110-0492, SW1 EVQ-P0E07K, SW2 EVQ-P0E07K

Commit message: Update Trigger Module
Other:
- board text removed: "Designed by Mitch @ HHL"
- board text removed: "ProGCC 4"

Commit message: Main Board/Trigger Board Update
- Main board updated with Kailh tactile switches
- Trigger board updated with Kailh tactile switches
- USBW board updated to remove unneeded diode, move position of USB-C port
Parts:
- SW1, SW2: value EVQ-P0E07K -> CMI624301D09
Changed lines of the file:
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@@
 			)
 		)
-		(property "Value" "EVQ-P0E07K"
+		(property "Value" "CMI624301D09"
 			(at 0 1 0)
 			(unlocked yes)
@@
 			)
 		)
-		(property "Datasheet" ""
+		(property "Datasheet" "~"
 			(at 0 0 0)
 			(unlocked yes)
@@
 			)
 		)
-		(property "MPN" "EVQ-P0E07K"
+		(property "MPN" "CMI624301D09"
 			(at 0 0 0)
 			(unlocked yes)
@@
 			)
 		)
-		(property "LCSC" "C395225"
+		(property "LCSC" ""
 			(at 0 0 0)
 			(unlocked yes)
@@
 			)
 		)
-		(property "Manufacturer" "PANASONIC"
+		(property "Manufacturer" "Kailh"
 			(at 0 0 0)
 			(unlocked yes)
@@
 			)
 		)
-		(sheetname "Root")
+		(sheetname "/")
 		(sheetfile "PGS_Trigger_Board.kicad_sch")
 		(attr through_hole)
@@
 			)
 		)
-		(property "Datasheet" ""
+		(property "Datasheet" "~"
 			(at 0 0 90)
 			(unlocked yes)
@@
 		)
 		(property ki_fp_filters "Connector*:*_1x??_*")
-		(sheetname "Root")
+		(sheetname "/")
 		(sheetfile "PGS_Trigger_Board.kicad_sch")
 		(attr smd)
@@
 			)
 		)
-		(property "Value" "EVQ-P0E07K"
+		(property "Value" "CMI624301D09"
 			(at 0 1 180)
 			(unlocked yes)
@@
 			)
 		)
-		(property "Datasheet" ""
+		(property "Datasheet" "https://uelectronics.com/wp-content/uploads/2024/12/Datasheet-Microinterruptor-Silencioso-para-Mouse-CMI624301D09.pdf?srsltid=AfmBOop6n-LI93civhddjTPUOZCj3iSyUFg8_0Vf9y402ymvABNEZW8f"
 			(at 0 0 180)
 			(unlocked yes)
@@
 			)
 		)
-		(property "MPN" "EVQ-P0E07K"
+		(property "MPN" "CMI624301D09"
 			(at 0 0 180)
 			(unlocked yes)
@@
 			)
 		)
-		(property "LCSC" "C395225"
+		(property "LCSC" ""
 			(at 0 0 180)
 			(unlocked yes)
@@
 			)
 		)
-		(property "Manufacturer" "PANASONIC"
+		(property "Manufacturer" "Kailh"
 			(at 0 0 180)
 			(unlocked yes)
@@
 			)
 		)
-		(sheetname "Root")
+		(sheetname "/")
 		(sheetfile "PGS_Trigger_Board.kicad_sch")
 		(attr through_hole)
