File: PCB/Projects/Main Board/PGS_Main_Board.kicad_pcb (KiCad board)
At the start: 4 copper layers, 109.9 x 60.8 mm, 119 parts, among them J1 SM02B-SURS-TF_LF__SN_, J2 SM02B-SURS-TF_LF__SN_, J3 Molex 505110-0892, J5 Molex 505110-0892, J6 Molex 505110-0492, J7 Molex 505110-0492, J8 Conn_01x04_Pin, J9 Molex 505110-1792, Q1 MMBT2222A, Q2 MMBT2222A, SW1 TS-1187A-C-A-B, SW14 CMI627301D60, SW15 TS-1187A-C-A-B, SW16 TS-1187A-C-A-B, SW2 TS-1187A-C-A-B, SW3 TS-1187A-C-A-B, SW4 TS-1187A-C-A-B, SW9 CMI627301D60, U1 RP2040, U3 GD25Q80EEIGR, U4 ST_LSM6, U5 ST_LSM6, Y1 ABM8-272-T3

Commit message: Sept 2026 Changes
Parts:
- removed C20, C21, C28: 100nF, Capacitor_SMD:C_0201_0603Metric
- removed C22: 1uF, Capacitor_SMD:C_0201_0603Metric
- removed D11, D12, D13, D14, D15, D16, D8, D9: BAS16VY,115, Package_TO_SOT_SMD:SOT-363_SC-70-6
- removed J6: Molex 505110-0492, hhl:5051100492
- removed R2: 10k, Resistor_SMD:R_0201_0603Metric
- removed S1: TMUX1204DQAR, hhl:TMUX1204DQAR
- removed SW1, SW15, SW16, SW2: TS-1187A-C-A-B, hhl:TS-1187A-C-E-B
- removed SW12, SW13: ~, hhl:pgs_abxy
- removed SW14: CMI627301D60, hhl:EVQP0
- added C17: 100n, Capacitor_SMD:C_0201_0603Metric, B.Cu at (37.7, 58.6)
- added C19: 100n, Capacitor_SMD:C_0201_0603Metric, F.Cu at (20.9, -9.32)
- added C29: 100n, Capacitor_SMD:C_0201_0603Metric, F.Cu at (20.9, -7.58)
- added C30: 100n, Capacitor_SMD:C_0201_0603Metric, F.Cu at (20.9, -5.83)
- added C31: 100n, Capacitor_SMD:C_0201_0603Metric, F.Cu at (20.9, -4.08)
- added C32: 100n, Capacitor_SMD:C_0201_0603Metric, F.Cu at (23.4, -9.32)
- added C33: 100n, Capacitor_SMD:C_0201_0603Metric, F.Cu at (23.4, -7.58)
- added C34: 100n, Capacitor_SMD:C_0201_0603Metric, F.Cu at (23.4, -5.83)
- added C35: 100n, Capacitor_SMD:C_0201_0603Metric, F.Cu at (23.4, -4.08)
- added C36: 100n, Capacitor_SMD:C_0201_0603Metric, F.Cu at (25.9, -9.32)
- added C37: 100n, Capacitor_SMD:C_0201_0603Metric, F.Cu at (25.9, -7.58)
- added C38: 100n, Capacitor_SMD:C_0201_0603Metric, F.Cu at (25.9, -5.83)
- added C39: 4.7u, Capacitor_SMD:C_0402_1005Metric, B.Cu at (77.3, 31.2)
- added C40: 4.7u, Capacitor_SMD:C_0402_1005Metric, B.Cu at (78.0, 31.8)
- added C41: 4.7u, Capacitor_SMD:C_0402_1005Metric, B.Cu at (79.0, 29.4)
- added J10: Conn_01x04_Pin, Connector_PinHeader_2.00mm:PinHeader_1x04_P2.00mm_Vertical, F.Cu at (33.9, -20.3)
- added J11: Molex 505110-0592, hhl:5051100592, B.Cu at (57.3, 24.3)
- added L1: 3.3u, hhl:L_pol_2016, B.Cu at (79.3, 32.7)
- added R23: 100R, Resistor_SMD:R_0201_0603Metric, F.Cu at (25.9, -4.08)
- added R31: 27R, Resistor_SMD:R_0201_0603Metric, F.Cu at (28.3, -9.32)
- added R32: 27R, Resistor_SMD:R_0201_0603Metric, F.Cu at (28.3, -7.58)
- added R33: 27R, Resistor_SMD:R_0201_0603Metric, F.Cu at (28.3, -5.83)
- added R34: 27R, Resistor_SMD:R_0201_0603Metric, F.Cu at (28.3, -4.08)
- added U10: HAL4395, hhl:SOT-23-5L, B.Cu at (39.8, 58.6)
- added U11: HAL4395, hhl:SOT-23-5L, B.Cu at (56.3, 58.6)
- added U2: RP2350_80QFN, hhl:RP2350-QFN-80-1EP_10x10_P0.4mm_EP3.4x3.4mm_ThermalVias, B.Cu at (70.8, 29.1)
- added U6: HAL4395, hhl:SOT-23-5L, B.Cu at (123.7, 37.2)
- added U7: HAL4395, hhl:SOT-23-5L, B.Cu at (99.9, 37.2)
- added U8: HAL4395, hhl:SOT-23-5L, B.Cu at (48.0, 50.3)
- added U9: HAL4395, hhl:SOT-23-5L, B.Cu at (48.0, 66.8)
- C18: value 1uF -> 100n
- C23: value 100nF -> 4.7u; footprint Capacitor_SMD:C_0201_0603Metric -> Capacitor_SMD:C_0402_1005Metric
- C3, C4, C5, C6, C7, C8: value 100nF -> 100n
- J7: value Molex 505110-0492 -> Molex 505110-0452; footprint hhl:5051100492 -> hhl:5051100592
- R11: value 100R -> 33
- R12, R13, R14, R16, R17, R18, R19, R20, R21, R22, R24, R30: value 100R -> 27R
- R15: value 100R -> 1k
- R25: value 1k -> 27R
- SW10: value ~ -> SW_Push; footprint hhl:pgs_abxy -> hhl:KSC-TE; moved to B.Cu
- SW11: value ~ -> SW_Push; footprint hhl:pgs_abxy -> hhl:KSC-TE
- SW3, SW4: value TS-1187A-C-A-B -> SW_Push; footprint hhl:TS-1187A-C-E-B -> hhl:KSC-TE
- SW5, SW6, SW7, SW8: value ~ -> SW_Push; footprint hhl:pgs_dpad -> hhl:KSC-TE
- SW9: value CMI627301D60 -> SW_Push; footprint hhl:EVQP0 -> hhl:KSC-TE
- U1: value RP2040 -> HAL4395; footprint Package_DFN_QFN:QFN-56-1EP_7x7mm_P0.4mm_EP3.2x3.2mm -> hhl:SOT-23-5L
- U3: value GD25Q80EEIGR -> HAL4395; footprint hhl:USON-8-EP(2x3) -> hhl:SOT-23-5L
- moved SW11 61.4 mm to (70.8, 68.4)
- moved C5 59.0 mm to (123.7, 39.3), turned to 0 degrees
- moved C8 48.2 mm to (50.1, 66.8), turned to 90 degrees
- moved C4 47.8 mm to (114.2, 47.7), turned to -90 degrees
- moved SW8 44.7 mm to (70.8, 29.1), turned to 0 degrees
- moved U1 40.9 mm to (111.8, 26.9), turned to 180 degrees
- moved U3 40.9 mm to (111.8, 47.5), turned to 0 degrees
- moved C7 36.5 mm to (50.1, 50.3), turned to 90 degrees
- moved C3 36.3 mm to (111.8, 29.0), turned to 0 degrees
- moved SW10 35.7 mm to (114.8, 62.5), turned to 180 degrees
- moved C18 34.6 mm to (58.4, 58.6), turned to 90 degrees
- moved SW5 33.9 mm to (79.8, 37.6), turned to 90 degrees
- moved SW6 30.9 mm to (61.8, 37.6)
- moved R22 26.2 mm to (37.5, 26.8)
- moved SW4 25.7 mm to (56.8, 26.1), turned to 0 degrees
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Connections:
- C18 pad 1: GND -> +3V3
- C18 pad 2: +1V1 -> GND
- C23 pad 1: +3V3 -> +1V1
- C3 pad 1: GND -> +3V3
- C3 pad 2: +1V1 -> GND
- C7 pad 1: GND -> +3V3
- C7 pad 2: +3V3 -> GND
- C8 pad 1: GND -> +3V3
- C8 pad 2: +3V3 -> GND
- J3 pad 7: G -> STICK_R_BTN_IN
- J5 pad 7: F -> STICK_L_BTN_IN
- J7 pad 1: G -> T_R_3V3
- J7 pad 4: G -> T_R_EN
- R11 pad 1: Net-(U1-GPIO10) -> +3V3
- R11 pad 2: A -> /VREG_AVDD
- R12 pad 1: Net-(U1-GPIO4) -> N_DATA_3.3
- R12 pad 2: N_DATA_3.3 -> Net-(U2-GPIO4)
- R13 pad 1: Net-(U1-GPIO5) -> N_LATCH_3.3
- R13 pad 2: N_LATCH_3.3 -> Net-(U2-GPIO5)
- R14 pad 1: Net-(U1-GPIO6) -> N_CLOCK_3.3
- R14 pad 2: N_CLOCK_3.3 -> Net-(U2-GPIO6)
- R15 pad 1: Net-(U1-GPIO19) -> Net-(U2-RUN)
- R15 pad 2: I -> unconnected-(R15-Pad2)
- R16 pad 1: Net-(U1-GPIO18) -> BTN_PWR
- R16 pad 2: H -> Net-(U2-GPIO9)
- R17 pad 1: Net-(U1-GPIO22) -> STICK_L_BTN_IN
- R17 pad 2: G -> Net-(U2-GPIO10)
- R18 pad 1: Net-(U1-GPIO15) -> GRIP_L_BTN
- R18 pad 2: F -> Net-(U2-GPIO11)
- R19 pad 1: Net-(U1-GPIO14) -> DPAD_EN
- R19 pad 2: E -> Net-(U2-GPIO13)
- R20 pad 1: Net-(U1-GPIO13) -> TRIGGER_EN_L
- R20 pad 2: D -> Net-(U2-GPIO14)
- R21 pad 1: Net-(U1-GPIO12) -> GRIP_R_BTN
- R21 pad 2: C -> Net-(U2-GPIO26)
- R22 pad 1: Net-(U1-GPIO11) -> MINUS_BTN
- R22 pad 2: B -> Net-(U2-GPIO16)
- R24 pad 1: Net-(U1-GPIO25) -> ABXY_EN
- R24 pad 2: RGB_OUT -> Net-(U2-GPIO27)
- R25 pad 1: USB_BOOT -> CAPTURE_BTN
- R25 pad 2: Net-(U3-/CS) -> Net-(U2-GPIO17)
- R30 pad 1: Net-(U1-GPIO9) -> HOME_BTN
- R30 pad 2: BTN_PWR -> Net-(U2-GPIO18)
- SW10 pad 1: I -> unconnected-(SW10-Pad1)
- SW10 pad 2: Net-(D16B-A) -> unconnected-(SW10-Pad2)
- SW11 pad 1: I -> GND
- SW11 pad 2: Net-(D16A-A) -> BTN_PWR
- SW5 pad 1: H -> unconnected-(SW5-Pad1)
- SW5 pad 2: Net-(D14A-A) -> unconnected-(SW5-Pad2)
- SW6 pad 1: H -> unconnected-(SW6-Pad1)
- SW6 pad 2: Net-(D13C-A) -> unconnected-(SW6-Pad2)
- SW7 pad 1: H -> unconnected-(SW7-Pad1)
- SW7 pad 2: Net-(D14B-A) -> unconnected-(SW7-Pad2)
- SW8 pad 1: H -> unconnected-(SW8-Pad1)
- SW8 pad 2: Net-(D13B-A) -> unconnected-(SW8-Pad2)
- SW9 pad 1: H -> unconnected-(SW9-Pad1)
- SW9 pad 2: Net-(D13A-A) -> unconnected-(SW9-Pad2)
- U1 pad 2: WL_ON -> ABXY_EN
- U1 pad 3: WL_D -> GND
- U1 pad 4: I2C1_SDA -> unconnected-(U1-NC-Pad4)
- U1 pad 5: I2C1_SCL -> ADC_0
- U3 pad 1: Net-(U3-/CS) -> +3V3
- U3 pad 2: SIO1 -> ABXY_EN
- U3 pad 3: SIO2 -> GND
- U3 pad 4: GND -> unconnected-(U3-NC-Pad4)
- U3 pad 5: SIO0 -> ADC_1
- U4 pad 1: GND -> SPI1_RX
- U4 pad 12: +3V3 -> IMU0_CS
- U4 pad 13: I2C0_SCL -> SPI1_CLK
- U4 pad 14: I2C0_SDA -> SPI1_TX
- U5 pad 1: +3V3 -> SPI1_RX
- U5 pad 12: +3V3 -> IMU1_CS
- U5 pad 13: I2C0_SCL -> SPI1_CLK
- U5 pad 14: I2C0_SDA -> SPI1_TX
Routing:
- net H: track 149.0 -> 0.00 mm, vias 9 -> 0
- net I: track 122.6 -> 0.00 mm, vias 5 -> 0
- net +3V3: track 97.8 -> 1.19 mm, vias 35 -> 0
- net GND: track 99.5 -> 4.50 mm, vias 55 -> 1
- net LRA_R: track 93.3 -> 0.00 mm, vias 7 -> 0
- net C: track 79.8 -> 0.00 mm, vias 2 -> 0
- net D: track 79.5 -> 0.00 mm, vias 2 -> 0
- net E: track 78.8 -> 0.00 mm, vias 2 -> 0
- net LRA_L: track 77.1 -> 0.00 mm, vias 3 -> 0
- net B: track 74.0 -> 0.00 mm, vias 2 -> 0
- net A: track 70.9 -> 0.00 mm, vias 2 -> 0
- net G: track 64.2 -> 0.00 mm, vias 3 -> 0
- net Net-(D15C-A): track 60.7 -> 0.00 mm, vias 2 -> 0
- net F: track 58.9 -> 0.00 mm, vias 2 -> 0
- net STICK_R_Y_OUT: track 55.7 -> 0.00 mm, vias 4 -> 0
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- removed copper zone on In1.Cu, net +3V3
- removed copper zone on B.Cu, net GND
- removed copper zone on F.Cu, net GND
- removed copper zone on In2.Cu, net GND
Other:
- board size 109.9 x 60.8 mm -> 109.5 x 60.7 mm

Commit message: Routing Changes
Parts:
- removed R23: 100R, Resistor_SMD:R_0201_0603Metric
- removed R27: 1k, Resistor_SMD:R_0201_0603Metric
- added R35: 27R, Resistor_SMD:R_0201_0603Metric, F.Cu at (7.70, -1.62)
- C19, C29, C30, C31, C32, C33, C34, C35, C36, C37, C38: moved to B.Cu
- R15, R26: value 1k -> 27R; moved to F.Cu
- R16, R17, R18, R21, R22, R25, R30: moved to F.Cu
- moved R24 81.5 mm to (28.3, -5.83)
- moved R33 81.5 mm to (102.3, 28.4), turned to 180 degrees
- moved R21 80.0 mm to (109.6, 61.3), turned to 90 degrees
- moved R26 79.1 mm to (7.70, -3.38), turned to 0 degrees
- moved C36 70.2 mm to (73.8, 41.9), turned to -90 degrees
- moved C32 68.8 mm to (78.5, 31.9), turned to 45 degrees
- moved C37 68.3 mm to (76.5, 38.3), turned to -45 degrees
- moved C31 67.2 mm to (78.1, 31.4), turned to 45 degrees
- moved C19 67.1 mm to (76.3, 28.5), turned to 45 degrees
- moved C30 65.4 mm to (67.8, 39.8), turned to -135 degrees
- moved R31 65.2 mm to (81.0, 29.1), turned to 180 degrees
- moved C29 64.3 mm to (65.4, 38.9), turned to -135 degrees
- moved C38 60.4 mm to (75.8, 28.0), turned to 45 degrees
- moved C35 58.1 mm to (64.7, 36.8), turned to -135 degrees
- moved C33 56.3 mm to (65.7, 29.6), turned to -135 degrees
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Connections:
- R15 pad 2: unconnected-(R15-Pad2) -> BTN_RUN
- R26 pad 1: +3V3 -> Net-(U2-QSPI_SS)
- R26 pad 2: I2C0_SCL -> BTN_BOOT
- SW10 pad 1: unconnected-(SW10-Pad1) -> GRIP_R_BTN
- SW10 pad 2: unconnected-(SW10-Pad2) -> GND
- SW11 pad 1: GND -> BTN_PWR
- SW11 pad 2: BTN_PWR -> GND
- SW3 pad 1: unconnected-(SW3-Pad1) -> PLUS_BTN
- SW3 pad 2: unconnected-(SW3-Pad2) -> GND
- SW4 pad 1: unconnected-(SW4-Pad1) -> MINUS_BTN
- SW4 pad 2: unconnected-(SW4-Pad2) -> GND
- SW5 pad 1: unconnected-(SW5-Pad1) -> HOME_BTN
- SW5 pad 2: unconnected-(SW5-Pad2) -> GND
- SW6 pad 1: unconnected-(SW6-Pad1) -> CAPTURE_BTN
- SW6 pad 2: unconnected-(SW6-Pad2) -> GND
- SW7 pad 1: unconnected-(SW7-Pad1) -> BTN_BOOT
- SW7 pad 2: unconnected-(SW7-Pad2) -> GND
- SW8 pad 1: unconnected-(SW8-Pad1) -> BTN_RUN
- SW8 pad 2: unconnected-(SW8-Pad2) -> GND
- SW9 pad 1: unconnected-(SW9-Pad1) -> GRIP_L_BTN
- SW9 pad 2: unconnected-(SW9-Pad2) -> GND
- U2 pad 75: USB_BOOT -> Net-(U2-QSPI_SS)
Routing:
- net +3V3: track 1.19 -> 71.8 mm, vias 0 -> 29
- net STICK_R_RGB_OUT: track 0.00 -> 62.5 mm, vias 0 -> 1
- net ADC_1: track 0.00 -> 53.1 mm, vias 0 -> 1
- net ADC_2: track 0.00 -> 44.9 mm, vias 0 -> 1
- net ADC_3: track 0.00 -> 44.1 mm, vias 0 -> 1
- net RGB_DPAD_IN: track 0.00 -> 43.0 mm, vias 0 -> 4
- net BTN_PWR: track 0.00 -> 34.3 mm, vias 0 -> 1
- net Net-(RGB5-DOUT): track 0.00 -> 28.3 mm, vias 0 -> 2
- net Net-(RGB3-DOUT): track 0.00 -> 26.2 mm, vias 0 -> 2
- net ADC_0: track 0.00 -> 25.8 mm, vias 0 -> 1
- net Net-(RGB1-DOUT): track 0.00 -> 21.1 mm
- net I2C1_SDA: track 0.00 -> 20.8 mm, vias 0 -> 1
- net I2C1_SCL: track 0.00 -> 20.0 mm, vias 0 -> 1
- net T_L_OUT: track 0.00 -> 19.6 mm
- net D-: track 0.00 -> 19.4 mm
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Other:
- board text added: "RESET"
- board text removed: "A"
- board text removed: "B"
- board text removed: "MUX"
- board text removed: "X"
- board text removed: "Y"

Commit message: PCB Routing
Parts:
- removed J10: Conn_01x04_Pin, Connector_PinHeader_2.00mm:PinHeader_1x04_P2.00mm_Vertical
- removed R19, R20, R24, R32, R35: 27R, Resistor_SMD:R_0201_0603Metric
- moved R26 78.4 mm to (75.6, 35.8), turned to 90 degrees
- moved R34 75.0 mm to (94.7, 30.8), turned to 180 degrees
- moved R21 10.2 mm to (119.7, 60.2)
- moved R15 6.79 mm to (66.0, 27.5), turned to 90 degrees
- moved R31 6.01 mm to (81.3, 23.1)
- moved J8 5.99 mm to (67.9, 14.8), turned to -90 degrees
- moved R17 5.18 mm to (60.1, 46.9), turned to 90 degrees
- moved R22 5.00 mm to (60.0, 29.2), turned to 0 degrees
- moved C1 1.80 mm to (61.2, 27.6)
- moved C2 1.80 mm to (64.8, 24.0)
- moved R1 1.80 mm to (65.6, 27.2)
- moved C23 1.80 mm to (66.8, 26.2)
- moved Y1 1.80 mm to (63.6, 26.3)
- moved J11 1.75 mm to (56.8, 22.3)
- moved J7 0.97 mm to (84.2, 22.3)
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Connections:
- net SPI1_RX renamed SPI0_RX
- J11 pad 1: T_L_3V3 -> +3V3
- J11 pad 2: T_L_OUT -> ADC_1
- J11 pad 3: T_ZL_OUT -> ADC_0
- J11 pad 5: T_L_GND -> GND
- J3 pad 8: STICK_R_BTN_OUT -> GND
- J5 pad 8: STICK_L_BTN_OUT -> GND
- J7 pad 1: T_R_3V3 -> +3V3
- J7 pad 2: T_R_OUT -> ADC_3
- J7 pad 3: T_ZR_OUT -> ADC_2
- J7 pad 5: T_R_GND -> GND
- J8 pad 4: VBUS_SYS -> +3V3
- R17 pad 2: Net-(U2-GPIO10) -> Net-(U2-GPIO13)
- R18 pad 2: Net-(U2-GPIO11) -> Net-(U2-GPIO10)
- R21 pad 2: Net-(U2-GPIO26) -> Net-(U2-GPIO32)
- R25 pad 2: Net-(U2-GPIO17) -> Net-(U2-GPIO15)
- R30 pad 2: Net-(U2-GPIO18) -> Net-(U2-GPIO30)
- R31 pad 2: Net-(U2-GPIO19) -> Net-(U2-GPIO29)
- R33 pad 2: Net-(U2-GPIO28) -> Net-(U2-GPIO35)
- R34 pad 2: Net-(U2-GPIO29) -> Net-(U2-GPIO33)
- U1 pad 5: ADC_0 -> ADC_2
- U10 pad 5: ADC_2 -> ADC_3
- U11 pad 5: ADC_3 -> ADC_0
- U2 pad 11: LRA_L -> DPAD_EN
- U2 pad 13: Net-(U2-GPIO14) -> T_L_EN
- U2 pad 14: IMU0_CS -> Net-(U2-GPIO15)
- U2 pad 17: Net-(U2-GPIO17) -> IMU0_CS
- U2 pad 18: Net-(U2-GPIO18) -> SPI0_CLK
- U2 pad 19: Net-(U2-GPIO19) -> SPI0_TX
- U2 pad 22: SPI1_CLK -> unconnected-(U2-GPIO22-Pad22)
- U2 pad 23: SPI1_TX -> unconnected-(U2-GPIO23-Pad23)
- U2 pad 25: Net-(U2-GPIO24) -> unconnected-(U2-GPIO24-Pad25)
- U2 pad 26: LRA_R -> unconnected-(U2-GPIO25-Pad26)
- U2 pad 27: Net-(U2-GPIO26) -> unconnected-(U2-GPIO26-Pad27)
- U2 pad 28: Net-(U2-GPIO27) -> unconnected-(U2-GPIO27-Pad28)
- U2 pad 36: Net-(U2-GPIO28) -> T_R_EN
- U2 pad 38: unconnected-(U2-GPIO30-Pad38) -> Net-(U2-GPIO30)
- U2 pad 39: unconnected-(U2-GPIO31-Pad39) -> LRA_R
- U2 pad 40: unconnected-(U2-GPIO32-Pad40) -> Net-(U2-GPIO32)
- U2 pad 42: unconnected-(U2-GPIO33-Pad42) -> Net-(U2-GPIO33)
- U2 pad 43: unconnected-(U2-GPIO34-Pad43) -> ABXY_EN
- U2 pad 44: unconnected-(U2-GPIO35-Pad44) -> Net-(U2-GPIO35)
- U2 pad 48: Net-(U2-GPIO39) -> unconnected-(U2-GPIO39-Pad48)
- U2 pad 49: ADC_0 -> STICK_L_Y_OUT
- U2 pad 52: ADC_1 -> STICK_L_X_OUT
- U2 pad 53: ADC_2 -> ADC_0
- U2 pad 54: ADC_3 -> ADC_1
- U2 pad 55: STICK_R_Y_OUT -> ADC_2
- U2 pad 56: STICK_R_X_OUT -> ADC_3
- U2 pad 57: STICK_L_X_OUT -> STICK_R_X_OUT
- U2 pad 58: STICK_L_Y_OUT -> STICK_R_Y_OUT
- U2 pad 9: Net-(U2-GPIO11) -> LRA_L
- U4 pad 13: SPI1_CLK -> SPI0_CLK
- U4 pad 14: SPI1_TX -> SPI0_TX
- U5 pad 13: SPI1_CLK -> SPI0_CLK
- U5 pad 14: SPI1_TX -> SPI0_TX
- U6 pad 5: ADC_2 -> ADC_3
- U7 pad 5: ADC_3 -> ADC_0
- U8 pad 5: ADC_0 -> ADC_2
Routing:
- net GND: track 12.8 -> 116.4 mm, vias 4 -> 55
- net ADC_3: track 44.1 -> 141.2 mm, vias 1 -> 4
- net ABXY_EN: track 0.00 -> 92.6 mm, vias 0 -> 4
- net ADC_1: track 53.1 -> 141.7 mm, vias 1 -> 4
- net STICK_L_X_OUT: track 1.87 -> 87.8 mm, vias 0 -> 2
- net STICK_L_Y_OUT: track 2.05 -> 86.0 mm, vias 0 -> 2
- net LRA_R: track 1.59 -> 84.0 mm, vias 0 -> 2
- net Net-(U2-GPIO32): track 0.00 -> 81.0 mm, vias 0 -> 2
- net LRA_L: track 1.62 -> 80.3 mm, vias 0 -> 1
- net Net-(U2-GPIO10): track 0.00 -> 76.0 mm, vias 0 -> 1
- net ADC_0: track 25.8 -> 101.5 mm, vias 1 -> 4
- net ADC_2: track 44.9 -> 119.6 mm, vias 1 -> 4
- net DPAD_EN: track 0.00 -> 69.1 mm, vias 0 -> 2
- net SPI0_RX: track 0.00 -> 57.9 mm, vias 0 -> 3
- net SPI0_CLK: track 0.00 -> 55.2 mm, vias 0 -> 3
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- added copper zone on In2.Cu, net +3V3
- added copper zone on B.Cu, net GND
- added copper zone on F.Cu, net GND
- added copper zone on In1.Cu, net GND
Other:
- outline, holes or cut-outs redrawn
- board text added: "Hand Held Legend, LLC Designed By Mitch Cairns 9.21.2026"
- board text added: "RP2354B"
- board text removed: "FLASH"
- board text removed: "Hand Held Legend, LLC Designed By Mitch Cairns 7.20.2025"
- board text removed: "RP2040"
