File: PCB/Projects/Main Board/PGS_Main_Board.kicad_pcb (KiCad board)
At the start: 4 copper layers, 109.5 x 60.7 mm, 120 parts, among them J1 SM02B-SURS-TF_LF__SN_, J11 Molex 505110-0592, J2 SM02B-SURS-TF_LF__SN_, J3 Molex 505110-0892, J5 Molex 505110-0892, J7 Molex 505110-0452, J8 Conn_01x04_Pin, J9 Molex 505110-1792, Q1 MMBT2222A, Q2 MMBT2222A, SW10 SW_Push, SW11 SW_Push, SW3 SW_Push, SW4 SW_Push, SW5 SW_Push, SW6 SW_Push, SW7 SW_Push, SW8 SW_Push, SW9 SW_Push, U1 HAL4395, U10 HAL4395, U11 HAL4395, U2 RP2350_80QFN, U3 HAL4395, U4 ST_LSM6, U5 ST_LSM6, U6 HAL4395, U7 HAL4395, U8 HAL4395, U9 HAL4395, Y1 ABM8-272-T3

Commit message: Consolidate custom symbols, footprints and 3D models into repo library
Make the hardware repo self-contained instead of depending on the external
HHL-KiCad-Lib checkout and the missing progcc_v3 symbol library.

- New PCB/Libraries/ProGCC 4 Library.kicad_sym: the 12 custom symbols,
  extracted from the schematics' embedded caches (identical to what the
  boards use; duplicate hhl/progcc_v3 CUS08F30 merged)
- Library.pretty: add the 7 missing footprints and replace 9 that differed
  from the placed footprints with the hhl copies the boards match
- PCB/Libraries/3dmodels: STEP models previously referenced by absolute
  path into HHL-KiCad-Lib, now via ${KIPRJMOD}/../../Libraries/3dmodels
- Relink hhl:/progcc_v3:/RP2350_80QFN_minimal: references in all four
  schematics and PCBs to "ProGCC 4 Library"
- Project sym-lib-table and fp-lib-table for all four boards using
  ${KIPRJMOD}-relative paths (replaces Main's absolute fp-lib-table path)

No electrical change. ERC: lib_symbol_issues cleared (Main 70->49,
USBW 36->22, Stick 7->2, Trigger unchanged). DRC unchanged on all boards.

Co-Authored-By: Claude Opus 5.5 <noreply@anthropic.com>
Parts:
- J1, J2: footprint hhl:JST_SM02B-SURS-TF_LF__SN_ -> ProGCC 4 Library:JST_SM02B-SURS-TF_LF__SN_
- J11, J7: footprint hhl:5051100592 -> ProGCC 4 Library:5051100592
- J3, J5: footprint hhl:5051100892 -> ProGCC 4 Library:5051100892
- J9: footprint hhl:5051101792 -> ProGCC 4 Library:5051101792
- L1: footprint hhl:L_pol_2016 -> ProGCC 4 Library:L_pol_2016
- RGB1, RGB10, RGB11, RGB12, RGB13, RGB14, RGB15, RGB16, RGB2, RGB3, RGB4, RGB5, RGB6, RGB7, RGB8, RGB9: footprint hhl:SK6805-EC-10 -> ProGCC 4 Library:SK6805-EC-10
- SW10, SW11, SW3, SW4, SW5, SW6, SW7, SW8, SW9: footprint hhl:KSC-TE -> ProGCC 4 Library:KSC-TE
- U1, U10, U11, U3, U6, U7, U8, U9: footprint hhl:SOT-23-5L -> ProGCC 4 Library:SOT-23-5L
- U2: footprint hhl:RP2350-QFN-80-1EP_10x10_P0.4mm_EP3.4x3.4mm_ThermalVias -> ProGCC 4 Library:RP2350-QFN-80-1EP_10x10_P0.4mm_EP3.4x3.4mm_ThermalVias
- U4, U5: footprint hhl:LGA14 -> ProGCC 4 Library:LGA14
Changed lines of the file:
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@@
 		)
 	)
-	(footprint "hhl:SK6805-EC-10"
+	(footprint "ProGCC 4 Library:SK6805-EC-10"
 		(layer "F.Cu")
 		(at 111.752734 30.929086)
@@
 		)
 	)
-	(footprint "hhl:SK6805-EC-10"
+	(footprint "ProGCC 4 Library:SK6805-EC-10"
 		(layer "F.Cu")
 		(at 72.293091 51.211695)
@@
 		)
 	)
-	(footprint "hhl:SK6805-EC-10"
+	(footprint "ProGCC 4 Library:SK6805-EC-10"
 		(layer "F.Cu")
 		(at 111.752734 51.504086)
@@
 		)
 	)
-	(footprint "hhl:SK6805-EC-10"
+	(footprint "ProGCC 4 Library:SK6805-EC-10"
 		(layer "F.Cu")
 		(at 111.752734 43.504086)
@@
 		)
 	)
-	(footprint "hhl:SK6805-EC-10"
+	(footprint "ProGCC 4 Library:SK6805-EC-10"
 		(layer "F.Cu")
 		(at 48.03883 53.884448)
@@
 		)
 	)
-	(footprint "hhl:KSC-TE"
+	(footprint "ProGCC 4 Library:KSC-TE"
 		(layer "F.Cu")
 		(at 70.784037 29.138316)
@@
 		)
 	)
-	(footprint "hhl:KSC-TE"
+	(footprint "ProGCC 4 Library:KSC-TE"
 		(layer "F.Cu")
 		(at 56.772471 26.132897 180)
@@
 		)
 	)
-	(footprint "hhl:SK6805-EC-10"
+	(footprint "ProGCC 4 Library:SK6805-EC-10"
 		(layer "F.Cu")
 		(at 99.852734 33.216586)
@@
 		)
 	)
-	(footprint "hhl:SK6805-EC-10"
+	(footprint "ProGCC 4 Library:SK6805-EC-10"
 		(layer "F.Cu")
 		(at 48.03883 63.284448)
@@
 		)
 	)
-	(footprint "hhl:KSC-TE"
+	(footprint "ProGCC 4 Library:KSC-TE"
 		(layer "F.Cu")
 		(at 70.784037 37.412061)
@@
 		)
 	)
-	(footprint "hhl:SK6805-EC-10"
+	(footprint "ProGCC 4 Library:SK6805-EC-10"
 		(layer "F.Cu")
 		(at 52.73883 58.584448)
@@
 		)
 	)
-	(footprint "hhl:KSC-TE"
+	(footprint "ProGCC 4 Library:KSC-TE"
 		(layer "F.Cu")
 		(at 84.795603 26.132897)
@@
 		)
 	)
-	(footprint "hhl:KSC-TE"
+	(footprint "ProGCC 4 Library:KSC-TE"
 		(layer "F.Cu")
 		(at 61.772471 37.632897 90)
@@
 		)
 	)
-	(footprint "hhl:SK6805-EC-10"
+	(footprint "ProGCC 4 Library:SK6805-EC-10"
 		(layer "F.Cu")
 		(at 64.793092 51.211695)
@@
 		)
 	)
-	(footprint "hhl:SK6805-EC-10"
+	(footprint "ProGCC 4 Library:SK6805-EC-10"
 		(layer "F.Cu")
 		(at 99.852734 41.216586)
@@
 		)
 	)
-	(footprint "hhl:SK6805-EC-10"
+	(footprint "ProGCC 4 Library:SK6805-EC-10"
 		(layer "F.Cu")
 		(at 111.752734 22.929086)
@@
 		)
 	)
-	(footprint "hhl:KSC-TE"
+	(footprint "ProGCC 4 Library:KSC-TE"
 		(layer "F.Cu")
 		(at 79.795603 37.632897 -90)
@@
 		)
 	)
-	(footprint "hhl:SK6805-EC-10"
+	(footprint "ProGCC 4 Library:SK6805-EC-10"
 		(layer "F.Cu")
 		(at 123.652734 41.216586)
@@
 		)
 	)
-	(footprint "hhl:KSC-TE"
+	(footprint "ProGCC 4 Library:KSC-TE"
 		(layer "F.Cu")
 		(at 70.772471 68.382897)
@@
 		)
 	)
-	(footprint "hhl:SK6805-EC-10"
+	(footprint "ProGCC 4 Library:SK6805-EC-10"
 		(layer "F.Cu")
 		(at 76.043093 51.211695)
@@
 		)
 	)
-	(footprint "hhl:SK6805-EC-10"
+	(footprint "ProGCC 4 Library:SK6805-EC-10"
 		(layer "F.Cu")
 		(at 123.652734 33.216586)
@@
 		)
 	)
-	(footprint "hhl:SK6805-EC-10"
+	(footprint "ProGCC 4 Library:SK6805-EC-10"
 		(layer "F.Cu")
 		(at 43.338832 58.584448)
@@
 		)
 	)
-	(footprint "hhl:SK6805-EC-10"
+	(footprint "ProGCC 4 Library:SK6805-EC-10"
 		(layer "F.Cu")
 		(at 68.543091 51.211695)
@@
 		)
 	)
-	(footprint "hhl:5051100892"
+	(footprint "ProGCC 4 Library:5051100892"
 		(layer "B.Cu")
 		(at 47.15 58.075 180)
@@
 		)
 	)
-	(footprint "hhl:SOT-23-5L"
+	(footprint "ProGCC 4 Library:SOT-23-5L"
 		(layer "B.Cu")
 		(at 123.652734 37.216586 180)
@@
 		)
 	)
-	(footprint "hhl:KSC-TE"
+	(footprint "ProGCC 4 Library:KSC-TE"
 		(layer "B.Cu")
 		(at 114.761814 62.529128 180)
@@
 		)
 	)
-	(footprint "hhl:KSC-TE"
+	(footprint "ProGCC 4 Library:KSC-TE"
 		(layer "B.Cu")
 		(at 26.80626 62.529128 180)
@@
 		)
 	)
-	(footprint "hhl:SOT-23-5L"
+	(footprint "ProGCC 4 Library:SOT-23-5L"
 		(layer "B.Cu")
 		(at 48.03883 66.834448 -90)
@@
 		)
 	)
-	(footprint "hhl:JST_SM02B-SURS-TF_LF__SN_"
+	(footprint "ProGCC 4 Library:JST_SM02B-SURS-TF_LF__SN_"
 		(layer "B.Cu")
 		(at 111.975 67.925 180)
@@
 		)
 	)
-	(footprint "hhl:LGA14"
+	(footprint "ProGCC 4 Library:LGA14"
 		(layer "B.Cu")
 		(at 57.25 16.825 180)
@@
 		)
 	)
-	(footprint "hhl:LGA14"
+	(footprint "ProGCC 4 Library:LGA14"
 		(layer "B.Cu")
 		(at 82.9 16.825 180)
@@
 		)
 	)
-	(footprint "hhl:SOT-23-5L"
+	(footprint "ProGCC 4 Library:SOT-23-5L"
 		(layer "B.Cu")
 		(at 111.752734 26.929086 180)
@@
 		)
 	)
-	(footprint "hhl:5051100592"
+	(footprint "ProGCC 4 Library:5051100592"
 		(layer "B.Cu")
 		(at 56.775 22.299999)
@@
 		)
 	)
-	(footprint "hhl:SOT-23-5L"
+	(footprint "ProGCC 4 Library:SOT-23-5L"
 		(layer "B.Cu")
 		(at 39.78883 58.584448 -90)
@@
 		)
 	)
-	(footprint "hhl:5051100592"
+	(footprint "ProGCC 4 Library:5051100592"
 		(layer "B.Cu")
 		(at 84.25 22.299999)
@@
 		)
 	)
-	(footprint "hhl:RP2350-QFN-80-1EP_10x10_P0.4mm_EP3.4x3.4mm_ThermalVias"
+	(footprint "ProGCC 4 Library:RP2350-QFN-80-1EP_10x10_P0.4mm_EP3.4x3.4mm_ThermalVias"
 		(layer "B.Cu")
 		(at 70.8 33.297225 45)
@@
 		)
 	)
-	(footprint "hhl:L_pol_2016"
+	(footprint "ProGCC 4 Library:L_pol_2016"
 		(layer "B.Cu")
 		(at 79.290963 36.833909 45)
@@
 		)
 	)
-	(footprint "hhl:SOT-23-5L"
+	(footprint "ProGCC 4 Library:SOT-23-5L"
 		(layer "B.Cu")
 		(at 56.28883 58.584448 -90)
@@
 		)
 	)
-	(footprint "hhl:SOT-23-5L"
+	(footprint "ProGCC 4 Library:SOT-23-5L"
 		(layer "B.Cu")
 		(at 99.852734 37.216586 180)
@@
 		)
 	)
-	(footprint "hhl:5051101792"
+	(footprint "ProGCC 4 Library:5051101792"
 		(layer "B.Cu")
 		(at 67.059 51.55)
@@
 		)
 	)
-	(footprint "hhl:JST_SM02B-SURS-TF_LF__SN_"
+	(footprint "ProGCC 4 Library:JST_SM02B-SURS-TF_LF__SN_"
 		(layer "B.Cu")
 		(at 30.975 68.175 180)
@@
 		)
 	)
-	(footprint "hhl:SOT-23-5L"
+	(footprint "ProGCC 4 Library:SOT-23-5L"
 		(layer "B.Cu")
 		(at 48.03883 50.334448 -90)
@@
 		)
 	)
-	(footprint "hhl:5051100892"
+	(footprint "ProGCC 4 Library:5051100892"
 		(layer "B.Cu")
 		(at 112.45 40.625 -90)
@@
 		)
 	)
-	(footprint "hhl:SOT-23-5L"
+	(footprint "ProGCC 4 Library:SOT-23-5L"
 		(layer "B.Cu")
 		(at 111.752734 47.504086 180)

Commit message: Main PCB: update from schematic
Fields and pin types only; no footprints, tracks, vias, zones or nets
changed (120 footprints, identical reference list and pad nets).

- HAL4395 description and tri-state OUT pin type on the 8 halls.
- Pin types synced (RP2354B NC pins, IMU power pins, RGB DOUT).
- R9/R10 Link corrected to the 10R part.
- Stale PCB data synced from schematic: R15/R26 MPN/LCSC (27R),
  J7 value 505110-0592, J7/J11 LCSC.
- Empty legacy fields removed.

DRC 238 -> 223 (the 15 schematic-parity mismatches cleared; all other
categories unchanged).

Co-Authored-By: Claude Opus 5.5 <noreply@anthropic.com>
Parts:
- J7: value Molex 505110-0452 -> Molex 505110-0592
