File: PCB/Projects/Main Board/PGS_Main_Board.kicad_pcb (KiCad board)
At the start: 4 copper layers, 109.5 x 60.7 mm, 120 parts, among them J1 SM02B-SURS-TF_LF__SN_, J11 Molex 505110-0592, J2 SM02B-SURS-TF_LF__SN_, J3 Molex 505110-0892, J5 Molex 505110-0892, J7 Molex 505110-0592, J8 Conn_01x04_Pin, J9 Molex 505110-1792, Q1 MMBT2222A, Q2 MMBT2222A, SW10 SW_Push, SW11 SW_Push, SW3 SW_Push, SW4 SW_Push, SW5 SW_Push, SW6 SW_Push, SW7 SW_Push, SW8 SW_Push, SW9 SW_Push, U1 HAL4395, U10 HAL4395, U11 HAL4395, U2 RP2350_80QFN, U3 HAL4395, U4 ST_LSM6, U5 ST_LSM6, U6 HAL4395, U7 HAL4395, U8 HAL4395, U9 HAL4395, Y1 ABM8-272-T3

Commit message: Main PCB: refill zones, GND stubs for starved thermals, DRC exclusions
- Zones refilled (applies the JST haptics-pad pour clearance rule).
- Short GND tracks from C9, C12, C27, C37 to nearby GND pads / pour.
- DRC exclusions (all reviewed): SW9 pad 2 edge clearance (accepted),
  courtyard overlaps J3-U3, J5-U10, J11-Y1, C23-Y1, R1-Y1 (no body or
  pad clash), starved thermals C9 and C12.

DRC: 0 errors, no unconnected items.

Co-Authored-By: Claude Opus 5.5 <noreply@anthropic.com>
Routing:
- net GND: track 116.4 -> 121.5 mm
Changed lines of the file:
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@@
+	)
+	(segment
+		(start 30.117501 57.6)
+		(end 30.117501 57.986969)
+		(width 0.2)
+		(layer "F.Cu")
+		(net "GND")
 	)
 	(segment
@@
 	)
 	(segment
+		(start 32.12 65.37)
+		(end 32.12 65.9)
+		(width 0.2)
+		(layer "F.Cu")
+		(net "GND")
+	)
+	(segment
 		(start 123.317734 40.382266)
 		(end 123.675 40.025)
@@
 	)
 	(segment
+		(start 31.875 64.434247)
+		(end 31.875 65.125)
+		(width 0.2)
+		(layer "F.Cu")
+		(net "GND")
+	)
+	(segment
 		(start 52.40383 57.52883)
 		(end 51.825 56.95)
@@
 	)
 	(segment
+		(start 31.875 65.125)
+		(end 32.12 65.37)
+		(width 0.2)
+		(layer "F.Cu")
+		(net "GND")
+	)
+	(segment
 		(start 111.417734 51.169086)
 		(end 111.417734 50.607266)
@@
 	)
 	(segment
+		(start 29.842128 58.832873)
+		(end 29.662501 59.0125)
+		(width 0.2)
+		(layer "F.Cu")
+		(net "GND")
+	)
+	(segment
 		(start 81.895603 28.132897)
 		(end 80.017103 28.132897)
@@
 	)
 	(segment
+		(start 29.842128 58.262342)
+		(end 29.842128 58.832873)
+		(width 0.2)
+		(layer "F.Cu")
+		(net "GND")
+	)
+	(segment
 		(start 68.775 48.925)
 		(end 68.625 48.925)
@@
 	)
 	(segment
+		(start 30.117501 57.986969)
+		(end 29.842128 58.262342)
+		(width 0.2)
+		(layer "F.Cu")
+		(net "GND")
+	)
+	(segment
 		(start 87.695603 28.132897)
 		(end 89.557897 28.132897)
@@
 	)
 	(segment
+		(start 76.925 38.725)
+		(end 76.925 39.55)
+		(width 0.2)
+		(layer "B.Cu")
+		(net "GND")
+	)
+	(segment
 		(start 78.784785 31.623726)
 		(end 78.776274 31.623726)
@@
 	)
 	(segment
+		(start 82.97 14.9)
+		(end 83.805 14.9)
+		(width 0.2)
+		(layer "B.Cu")
+		(net "GND")
+	)
+	(segment
 		(start 79.469895 32.119895)
 		(end 80.15 32.8)
+		(width 0.2)
+		(layer "B.Cu")
+		(net "GND")
+	)
+	(segment
+		(start 76.701274 38.526274)
+		(end 76.726274 38.526274)
 		(width 0.2)
 		(layer "B.Cu")
@@
 		(width 0.2)
 		(layer "B.Cu")
+		(net "GND")
+	)
+	(segment
+		(start 76.726274 38.526274)
+		(end 76.925 38.725)
+		(width 0.2)
+		(layer "B.Cu")
