File: PCB/Projects/Main Board/PGS_Main_Board.kicad_sch (KiCad schematic)
At the start: 119 parts, among them J1 SM02B-SURS-TF_LF__SN_, J2 SM02B-SURS-TF_LF__SN_, J3 Molex 505110-0892, J5 Molex 505110-0892, J6 Molex 505110-0492, J7 Molex 505110-0492, J8 Conn_01x04_Pin, J9 Molex 505110-1792, Q1 MMBT2222A, Q2 MMBT2222A, SW1 TS-1187A-C-A-B, SW14 CMI627301D60, SW15 TS-1187A-C-A-B, SW16 TS-1187A-C-A-B, SW2 TS-1187A-C-A-B, SW3 TS-1187A-C-A-B, SW4 TS-1187A-C-A-B, SW9 CMI627301D60, U1 RP2040, U3 GD25Q80EEIGR, U4 ST_LSM6, U5 ST_LSM6, Y1 ABM8-272-T3

Commit message: Sept 2026 Changes
Parts:
- removed C20, C21, C28: 100nF, Capacitor_SMD:C_0201_0603Metric, symbol Device:C
- removed C22: 1uF, Capacitor_SMD:C_0201_0603Metric, symbol Device:C
- removed D11, D12, D13, D14, D15, D16, D8, D9: BAS16VY,115, Package_TO_SOT_SMD:SOT-363_SC-70-6, symbol progcc_v3:BAS16VY,115
- removed J6, J7: Molex 505110-0492, hhl:5051100492, symbol Connector:Conn_01x04_Pin
- removed R2: 10k, Resistor_SMD:R_0201_0603Metric, symbol Device:R_Small
- removed R25: 1k, Resistor_SMD:R_0201_0603Metric, symbol Device:R_Small
- removed S1: TMUX1204DQAR, hhl:TMUX1204DQAR, symbol hhl:TMUX1204DQAR
- removed SW1, SW15, SW16, SW2, SW3, SW4: TS-1187A-C-A-B, hhl:TS-1187A-C-E-B, symbol hhl:SW_TS-1187A
- removed SW12, SW13: ~, hhl:pgs_abxy, symbol Switch:SW_Push
- removed SW14: CMI627301D60, hhl:EVQP0, symbol Switch:SW_Push
- removed U1: RP2040, Package_DFN_QFN:QFN-56-1EP_7x7mm_P0.4mm_EP3.2x3.2mm, symbol progcc_v3:RP2040
- removed U3: GD25Q80EEIGR, hhl:USON-8-EP(2x3), symbol hhl:GD25Q80EEIGR
- added C17, C19, C29, C30, C31, C32, C33, C34, C35, C36, C37, C38: 100n, Capacitor_SMD:C_0201_0603Metric, symbol Device:C
- added C39, C40, C41: 4.7u, Capacitor_SMD:C_0402_1005Metric, symbol Device:C
- added J10: Conn_01x04_Pin, Connector_PinHeader_2.00mm:PinHeader_1x04_P2.00mm_Vertical, symbol Connector:Conn_01x04_Pin
- added J11: Molex 505110-0592, hhl:5051100592, symbol Connector:Conn_01x05_Pin
- added J7: Molex 505110-0452, hhl:5051100592, symbol Connector:Conn_01x05_Pin
- added L1: 3.3u, hhl:L_pol_2016, symbol Device:L
- added R23: 100R, Resistor_SMD:R_0201_0603Metric, symbol Device:R
- added R25, R31, R32, R33, R34: 27R, Resistor_SMD:R_0201_0603Metric, symbol Device:R
- added SW3, SW4: SW_Push, hhl:KSC-TE, symbol Switch:SW_Push
- added U1, U10, U11, U3, U6, U7, U8, U9: HAL4395, hhl:SOT-23-5L, symbol Regulator_Linear:TLV70012_SOT23-5
- added U2: RP2350_80QFN, hhl:RP2350-QFN-80-1EP_10x10_P0.4mm_EP3.4x3.4mm_ThermalVias, symbol hhl:RP2350_80QFN
- C18: value 1uF -> 100n; Confirmed YES -> (none); LCSC C76929 -> C76934; Link https://www.lcsc.com/product-detail/Multilayer-Ceramic-Capa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 -> (none); MPN GRM033R60J105KEA2D -> GRM033R61A104KE15D; Manufacturer Murata Electronics -> muRata; Package 0201 -> (none); Price 0.0007 -> (none); Reviewed Yes -> (none)
- C23: value 100nF -> 4.7u; footprint Capacitor_SMD:C_0201_0603Metric -> Capacitor_SMD:C_0402_1005Metric; LCSC C160831 -> C368809; MPN CL03A104KQ3NNNC -> CL05A475KP5NRNC; Package 0201 -> (none); Price 0.0007 -> (none); Reviewed Yes -> (none)
- C3, C4, C5, C7, C8: value 100nF -> 100n; Confirmed YES -> (none); LCSC C160831 -> C76934; Link https://www.lcsc.com/product-detail/Multilayer-Ceramic-Capa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 -> (none); MPN CL03A104KQ3NNNC -> GRM033R61A104KE15D; Manufacturer Samsung Electro-Mechanics -> muRata; Package 0201 -> (none); Price 0.0007 -> (none); Reviewed Yes -> (none)
- C6: value 100nF -> 100n; Confirmed YES -> (none); LCSC C160831 -> C76934; Link https://www.lcsc.com/product-detail/Multilayer-Ceramic-Capa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 -> (none); MPN CL03A104KQ3NNNC -> GRM033R61A104KE15D; Manufacturer Samsung Electro-Mechanics -> muRata; Package 0201 -> (none); Price 0.0015 -> (none); Reviewed Yes -> (none)
- R11: value 100R -> 33; Confirmed YES -> (none); LCSC C77623 -> C295794; Link https://www.lcsc.com/product-detail/Chip-Resistor-Surface-M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 -> (none); MPN RC0201FR-07100RL -> RC0201FR-0733RL; Package 0201 -> (none); Price 0.0006 -> (none); Reviewed Yes -> (none)
- R12, R13, R14, R16, R17, R18, R19, R20, R21, R22, R24, R30: value 100R -> 27R; LCSC C77623 -> C273268; MPN RC0201FR-07100RL -> RC0201FR-0727RL
- R15: value 100R -> 1k; Confirmed YES -> (none); LCSC C77623 -> C138165; Link https://www.lcsc.com/product-detail/Chip-Resistor-Surface-M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 -> (none); MPN RC0201FR-07100RL -> RC0201FR-071KL; Package 0201 -> (none); Price 0.0006 -> (none); Reviewed Yes -> (none)
- SW10, SW11: value ~ -> SW_Push; footprint hhl:pgs_abxy -> hhl:KSC-TE; LCSC (none) -> C221725; Link - -> (none); MPN (none) -> KSC201J LFS; Manufacturer (none) -> C&K; Package - -> (none); Price 0.082 -> (none); now fitted; now in the parts list
- SW5, SW6, SW7, SW8: value ~ -> SW_Push; footprint hhl:pgs_dpad -> hhl:KSC-TE; LCSC (none) -> C221725; Link - -> (none); MPN (none) -> KSC201J LFS; Manufacturer (none) -> C&K; Package - -> (none); Price 0.082 -> (none); now fitted; now in the parts list
- SW9: value CMI627301D60 -> SW_Push; footprint hhl:EVQP0 -> hhl:KSC-TE; LCSC (none) -> C221725; Link - -> (none); MPN CMI627301D60 -> KSC201J LFS; Manufacturer Kailh -> C&K; Package - -> (none); Price 0.082 -> (none); Reviewed Yes -> (none)
- T1, T2, T3, T4: value ~ -> (none)
- U4, U5: LCSC C784817 -> C126672; MPN LSM6DSRTR -> LSM6DSLTR
Connections:
- net +1V1: now also C23.1, C19.1, C29.1, C40.1, L1.1, U2.10 (DVDD), U2.32 (DVDD), U2.51 (DVDD), U2.65 (VREG_FB); no longer C18.2, C3.2
- net +3V3: now also C18.1, C3.1, C7.1, C8.1, R11.1, C17.1, C30.1, C31.1, C32.1, C33.1, C34.1, C35.1, C36.1, C37.1, C38.1, C39.1, U1.1 (VCC), U10.1 (VCC), U11.1 (VCC), U2.15 (IOVDD), U2.24 (IOVDD), U2.29 (IOVDD), U2.41 (IOVDD), U2.5 (IOVDD), U2.50 (IOVDD), U2.59 (ADC_AVDD), U2.60 (IOVDD), U2.64 (VREG_VIN), U2.68 (USB_OTP_VDD), U2.69 (QSPI_IOVDD), U2.76 (IOVDD), U3.1 (VCC), U6.1 (VCC), U7.1 (VCC), U8.1 (VCC), U9.1 (VCC); no longer C23.1, C7.2, C8.2, U4.12 (CS), U5.1 (SDO), U5.12 (CS)
- net BTN_PWR: now also R16.1, SW11.2, R23.2; no longer R30.2
- net DI+: now also U2.67 (USB_DP)
- net DI-: now also U2.66 (USB_DM)
- net GND: now also C18.2, C3.2, C7.2, C8.2, SW11.1, C17.2, C19.2, C29.2, C30.2, C31.2, C32.2, C33.2, C34.2, C35.2, C36.2, C37.2, C38.2, C39.2, C40.2, C41.2, J10.3 (Pin_3), U1.3 (GND), U10.3 (GND), U11.3 (GND), U2.62 (VREG_PGND), U2.81 (GND), U3.3 (GND), U6.3 (GND), U7.3 (GND), U8.3 (GND), U9.3 (GND); no longer C18.1, C3.1, C7.1, C8.1, U4.1 (SDO)
- net I2C0_SCL: no longer U4.13 (SCL), U5.13 (SCL)
- net I2C0_SDA: no longer U4.14 (SDA), U5.14 (SDA)
- net I2C1_SCL: now also U2.80 (GPIO3)
- net I2C1_SDA: now also U2.79 (GPIO2)
- net LRA_L: now also U2.11 (GPIO12)
- net LRA_R: now also U2.26 (GPIO25)
- net N_CLOCK_3.3: now also R14.1; no longer R14.2
- net N_DATA_3.3: now also R12.1; no longer R12.2
- net N_LATCH_3.3: now also R13.1; no longer R13.2
- net RGB_OUT: now also R33.1; no longer R24.2
- net STICK_L_X_OUT: now also U2.57 (GPIO46_ADC6)
- net STICK_L_Y_OUT: now also U2.58 (GPIO47_ADC7)
- net STICK_R_X_OUT: now also U2.56 (GPIO45_ADC5)
- net STICK_R_Y_OUT: now also U2.55 (GPIO44_ADC4)
- net SWCLK: now also J10.2 (Pin_2), U2.33 (SWCLK)
- net SWD: now also J10.1 (Pin_1), U2.34 (SWD)
- net T_L_OUT: now also J11.2 (Pin_2)
- net T_R_OUT: now also J7.2 (Pin_2)
- net T_ZL_OUT: now also J11.3 (Pin_3)
- net T_ZR_OUT: now also J7.3 (Pin_3)
- net USB_BOOT: now also U2.75 (QSPI_SS)
- net VBUS_SYS: now also J10.4 (Pin_4)
- net WL_CLK: now also U2.4 (GPIO7)
- net WL_CS: now also U2.6 (GPIO8)
- net WL_D: now also U2.78 (GPIO1)
- net WL_ON: now also U2.77 (GPIO0)
- net XTAL_IN: now also U2.30 (XIN)
- net XTAL_OUT: now also U2.31 (XOUT)
- net HOME_BTN: now reaches R30.1
- net MINUS_BTN: now reaches R22.1
- net GRIP_R_BTN: now reaches R21.1
- net TRIGGER_EN_L: now reaches R20.1
- net DPAD_EN: now reaches R19.1
- net DPAD_EN: now also U10.2 (~{EN}), U11.2 (~{EN}), U8.2 (~{EN}), U9.2 (~{EN})
- net GRIP_L_BTN: now reaches R18.1
- net at R15.1: now also U2.35 (RUN)
- net STICK_L_BTN_IN: now reaches R17.1
- net STICK_L_BTN_IN: now also J5.7 (Pin_7)
- net ABXY_EN: now reaches R24.1
- net ABXY_EN: now also U1.2 (~{EN}), U3.2 (~{EN}), U6.2 (~{EN}), U7.2 (~{EN})
- net A renamed VREG_AVDD
- net VREG_AVDD: now also C41.1, U2.61 (VREG_AVDD)
- net B: no longer names the net of R22.2
- net B: now also U2.16 (GPIO16)
- net C: no longer names the net of R21.2
- net C: now also U2.27 (GPIO26)
- net D: no longer names the net of R20.2
- net D: now also U2.13 (GPIO14)
- net E: no longer names the net of R19.2
- net E: now also U2.12 (GPIO13)
- net F: no longer names the net of R18.2
- net F: now also U2.9 (GPIO11); no longer J5.7 (Pin_7)
- net G: no longer names the net of R17.2
- net G: now also U2.8 (GPIO10); no longer J3.7 (Pin_7)
- removed net H: R16.2, SW5.1, SW6.1, SW7.1, SW8.1, SW9.1
- removed net I: R15.2, SW10.1, SW11.1
- new net: R12.2, U2.1 (GPIO4)
- new net: R25.2, U2.17 (GPIO17)
- new net: R30.2, U2.18 (GPIO18)
- new net: R31.2, U2.19 (GPIO19)
- new net: R13.2, U2.2 (GPIO5)
- new net: R32.2, U2.25 (GPIO24)
- new net: R24.2, U2.28 (GPIO27)
- new net: R14.2, U2.3 (GPIO6)
- new net: R33.2, U2.36 (GPIO28)
- new net: R34.2, U2.37 (GPIO29)
- new net: R23.1, U2.48 (GPIO39)
- new net: R16.2, U2.7 (GPIO9)
- new net ADC_0: U1.5 (OUT), U2.49 (GPIO40_ADC0), U8.5 (OUT)
- new net ADC_1: U2.52 (GPIO41_ADC1), U3.5 (OUT), U9.5 (OUT)
- new net ADC_2: U10.5 (OUT), U2.53 (GPIO42_ADC2), U6.5 (OUT)
- new net ADC_3: U11.5 (OUT), U2.54 (GPIO43_ADC3), U7.5 (OUT)
- new net CAPTURE_BTN: R25.1
- new net IMU0_CS: U2.14 (GPIO15), U4.12 (CS)
- new net IMU1_CS: U2.21 (GPIO21), U5.12 (CS)
- new net PLUS_BTN: R31.1
- new net SPI1_CLK: U2.22 (GPIO22), U4.13 (SCL), U5.13 (SCL)
- new net SPI1_RX: U2.20 (GPIO20), U4.1 (SDO), U5.1 (SDO)
- new net SPI1_TX: U2.23 (GPIO23), U4.14 (SDA), U5.14 (SDA)
- new net STICK_R_BTN_IN: J3.7 (Pin_7), R34.1
- new net TRIGGER_EN_R: R32.1
- new net T_L_3V3: J11.1 (Pin_1)
- new net T_L_EN: J11.4 (Pin_4)
- new net T_L_GND: J11.5 (Pin_5)
- new net T_R_3V3: J7.1 (Pin_1)
- new net T_R_EN: J7.4 (Pin_4)
- new net T_R_GND: J7.5 (Pin_5)
- new net VREG_LX: L1.2, U2.63 (VREG_LX)
Other:
- note added: "BOOTLOADER"
- note added: "DOWN"
- note added: "EAST"
- note added: "GRIP LEFT"
- note added: "GRIP RIGHT"
- note added: "LEFT"
- note added: "Make sure 27 ohm are close to RP2350"
- note added: "NORTH"
- note added: "PWM4 B"
- note added: "PWM6 A"
- note added: "RIGHT"
- note added: "RUN"
- note added: "SOUTH"
- note added: "UP"
- note added: "WEST"
- note removed: "1uF must be near pin 44"
- note removed: "1uF must be near pin 45"
- note removed: "Analog Mux"
- note removed: "CMI627301D60"
- note removed: "DDOWN"
- note removed: "DLEFT"
- note removed: "DRIGHT"
- note removed: "DUP"
- note removed: "EVQ-P0D07K for 130gf EVQ-P0E07K for 70gf"
- note removed: "Flash"
- note removed: "L Trigger"
- note removed: "LB"
- note removed: "R Trigger"
- note removed: "RB"
- note removed: "RP2040"
- note removed: "Stick Button L"
- note removed: "Stick Button R"
- note removed: "ZL Trigger"
- note removed: "ZR Trigger"

Commit message: Routing Changes
Parts:
- removed R23: 100R, Resistor_SMD:R_0201_0603Metric, symbol Device:R
- removed R27: 1k, Resistor_SMD:R_0201_0603Metric, symbol Device:R
- added R35: 27R, Resistor_SMD:R_0201_0603Metric, symbol Device:R
- R15: value 1k -> 27R; Confirmed (none) -> YES; LCSC C138165 -> C273268; Link (none) -> https://www.lcsc.com/product-detail/Chip-Resistor-Surface-M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; MPN RC0201FR-071KL -> RC0201FR-0727RL; Package (none) -> 0201; Price (none) -> 0.0006; Reviewed (none) -> Yes
- R26: value 1k -> 27R; Confirmed (none) -> YES; LCSC C138165 -> C273268; Link (none) -> https://www.lcsc.com/product-detail/Chip-Resistor-Surface-M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; MPN RC0201FR-071KL -> RC0201FR-0727RL
Connections:
- net I2C0_SCL is gone; now on net BTN_BOOT: R26.2
- net +3V3: no longer R26.1
- net BTN_PWR: now also SW11.1, R35.1; no longer SW11.2
- net CAPTURE_BTN: now also SW6.1
- net GND: now also SW10.2, SW11.2, SW3.2, SW4.2, SW5.2, SW6.2, SW7.2, SW8.2, SW9.2; no longer SW11.1
- net GRIP_L_BTN: now also SW9.1
- net GRIP_R_BTN: now also SW10.1
- net HOME_BTN: now also SW5.1
- net MINUS_BTN: now also SW4.1
- net PLUS_BTN: now also SW3.1
- net at U2.48 (GPIO39): now also R35.2
- net BTN_BOOT: now reaches SW7.1
- net BTN_RUN: now reaches SW8.1
- net BTN_RUN: now also R15.2
- net USB_BOOT: no longer names the net of U2.75 (QSPI_SS)
- net USB_BOOT: now also R26.1
Other:
- moved on the sheet: SW10, SW11, SW9

Commit message: PCB Routing
Parts:
- removed J10: Conn_01x04_Pin, Connector_PinHeader_2.00mm:PinHeader_1x04_P2.00mm_Vertical, symbol Connector:Conn_01x04_Pin
- removed R19, R20, R24, R32, R35: 27R, Resistor_SMD:R_0201_0603Metric, symbol Device:R
Connections:
- net T_L_3V3 is gone; now on net +3V3: J11.1 (Pin_1)
- net T_L_GND is gone; now on net GND: J11.5 (Pin_5)
- net T_L_OUT is gone; now on net ADC_1: J11.2 (Pin_2)
- net T_R_3V3 is gone; now on net +3V3: J7.1 (Pin_1)
- net T_R_GND is gone; now on net GND: J7.5 (Pin_5)
- net T_R_OUT is gone; now on net ADC_3: J7.2 (Pin_2)
- net T_ZL_OUT is gone; now on net ADC_0: J11.3 (Pin_3)
- net T_ZR_OUT is gone; now on net ADC_2: J7.3 (Pin_3)
- net VBUS_SYS is gone; now on net +3V3: J8.4 (Pin_4)
- net ABXY_EN: now also U2.43 (GPIO34)
- net ADC_0: now also U11.5 (OUT), U2.53 (GPIO42_ADC2), U7.5 (OUT); no longer U1.5 (OUT), U2.49 (GPIO40_ADC0), U8.5 (OUT)
- net ADC_1: now also U2.54 (GPIO43_ADC3); no longer U2.52 (GPIO41_ADC1)
- net ADC_2: now also U1.5 (OUT), U2.55 (GPIO44_ADC4), U8.5 (OUT); no longer U10.5 (OUT), U2.53 (GPIO42_ADC2), U6.5 (OUT)
- net ADC_3: now also U10.5 (OUT), U2.56 (GPIO45_ADC5), U6.5 (OUT); no longer U11.5 (OUT), U2.54 (GPIO43_ADC3), U7.5 (OUT)
- net DPAD_EN: now also U2.11 (GPIO12)
- net GND: now also J3.8 (Pin_8), J5.8 (Pin_8)
- net IMU0_CS: now also U2.17 (GPIO17); no longer U2.14 (GPIO15)
- net LRA_L: now also U2.9 (GPIO11); no longer U2.11 (GPIO12)
- net LRA_R: now also U2.39 (GPIO31); no longer U2.26 (GPIO25)
- net STICK_L_BTN_OUT: no longer J5.8 (Pin_8)
- net STICK_L_X_OUT: now also U2.52 (GPIO41_ADC1); no longer U2.57 (GPIO46_ADC6)
- net STICK_L_Y_OUT: now also U2.49 (GPIO40_ADC0); no longer U2.58 (GPIO47_ADC7)
- net STICK_R_BTN_OUT: no longer J3.8 (Pin_8)
- net STICK_R_X_OUT: now also U2.57 (GPIO46_ADC6); no longer U2.56 (GPIO45_ADC5)
- net STICK_R_Y_OUT: now also U2.58 (GPIO47_ADC7); no longer U2.55 (GPIO44_ADC4)
- net T_L_EN: now also U2.13 (GPIO14)
- net T_R_EN: now also U2.36 (GPIO28)
- net at U2.12 (GPIO13): now also R17.2
- net at R25.2: now also U2.14 (GPIO15); no longer U2.17 (GPIO17)
- net at R30.2: now also U2.38 (GPIO30); no longer U2.18 (GPIO18)
- net at R31.2: now also U2.37 (GPIO29); no longer U2.19 (GPIO19)
- net at U2.27 (GPIO26): no longer R21.2
- net at R33.2: now also U2.44 (GPIO35); no longer U2.36 (GPIO28)
- net at R34.2: now also U2.42 (GPIO33); no longer U2.37 (GPIO29)
- net at U2.40 (GPIO32): now also R21.2
- net at U2.8 (GPIO10): now also R18.2; no longer R17.2
- net SPI1_CLK renamed SPI0_CLK
- net SPI0_CLK: now also U2.18 (GPIO18); no longer U2.22 (GPIO22)
- net SPI1_RX renamed SPI0_RX
- net SPI1_TX renamed SPI0_TX
- net SPI0_TX: now also U2.19 (GPIO19); no longer U2.23 (GPIO23)
Other:
- note added: "PWM7 B"
- note removed: "PWM4 B"
- moved on the sheet: J8
