File: PCB/Projects/Main Board/PGS_Main_Board.kicad_sch (KiCad schematic)
At the start: 120 parts, among them J1 SM02B-SURS-TF_LF__SN_, J11 Molex 505110-0592, J2 SM02B-SURS-TF_LF__SN_, J3 Molex 505110-0892, J5 Molex 505110-0892, J7 Molex 505110-0452, J8 Conn_01x04_Pin, J9 Molex 505110-1792, Q1 MMBT2222A, Q2 MMBT2222A, SW10 SW_Push, SW11 SW_Push, SW3 SW_Push, SW4 SW_Push, SW5 SW_Push, SW6 SW_Push, SW7 SW_Push, SW8 SW_Push, SW9 SW_Push, U1 HAL4395, U10 HAL4395, U11 HAL4395, U2 RP2350_80QFN, U3 HAL4395, U4 ST_LSM6, U5 ST_LSM6, U6 HAL4395, U7 HAL4395, U8 HAL4395, U9 HAL4395, Y1 ABM8-272-T3

Commit message: Sync local board work; replace Trigger Board with Trigger FPC
- Update Main, Stick and USBW board layouts, schematics and 3D exports
- Replace the rigid Trigger Board project with the new Trigger FPC design
- Add shared PCB/Libraries footprint library and fp-lib-table
- Regenerate production outputs (gerbers, drills, placement, BOM) for all boards
- Stop tracking KiCad auto-backup folders and fp-info-cache; consolidate .gitignore

Co-Authored-By: Claude Opus 5 <noreply@anthropic.com>
Parts:
- J11: LCSC (none) -> C3168457
- J7: value Molex 505110-0452 -> Molex 505110-0592; LCSC (none) -> C3168457
- R1, R28, R29: LCSC C138165 -> (none); MPN RC0201FR-071KL -> (none)
- R10, R9: LCSC C106226 -> (none); MPN RC0201FR-0710RL -> (none)
- R11: LCSC C295794 -> (none); MPN RC0201FR-0733RL -> (none)
- R5, R6: LCSC C106225 -> (none); MPN RC0201FR-0710KL -> (none)
- R7, R8: LCSC C77623 -> (none); MPN RC0201FR-07100RL -> (none)
Other:
- note added: "PWM5 B"
- note removed: "PWM6 A"
- company: (none) -> Hand Held Legend LLC
- title: (none) -> PGC Super Main PCB
- moved on the sheet: C10, C11, C12, C13, C14, C19, C23, C29, C30, C31, C32, C33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
