File: PCB/Projects/Main Board/PGS_Main_Board.kicad_sch (KiCad schematic)
At the start: 120 parts, among them J1 SM02B-SURS-TF_LF__SN_, J11 Molex 505110-0592, J2 SM02B-SURS-TF_LF__SN_, J3 Molex 505110-0892, J5 Molex 505110-0892, J7 Molex 505110-0592, J8 Conn_01x04_Pin, J9 Molex 505110-1792, Q1 MMBT2222A, Q2 MMBT2222A, SW10 SW_Push, SW11 SW_Push, SW3 SW_Push, SW4 SW_Push, SW5 SW_Push, SW6 SW_Push, SW7 SW_Push, SW8 SW_Push, SW9 SW_Push, U1 HAL4395, U10 HAL4395, U11 HAL4395, U2 RP2350_80QFN, U3 HAL4395, U4 ST_LSM6, U5 ST_LSM6, U6 HAL4395, U7 HAL4395, U8 HAL4395, U9 HAL4395, Y1 ABM8-272-T3

Commit message: Consolidate custom symbols, footprints and 3D models into repo library
Make the hardware repo self-contained instead of depending on the external
HHL-KiCad-Lib checkout and the missing progcc_v3 symbol library.

- New PCB/Libraries/ProGCC 4 Library.kicad_sym: the 12 custom symbols,
  extracted from the schematics' embedded caches (identical to what the
  boards use; duplicate hhl/progcc_v3 CUS08F30 merged)
- Library.pretty: add the 7 missing footprints and replace 9 that differed
  from the placed footprints with the hhl copies the boards match
- PCB/Libraries/3dmodels: STEP models previously referenced by absolute
  path into HHL-KiCad-Lib, now via ${KIPRJMOD}/../../Libraries/3dmodels
- Relink hhl:/progcc_v3:/RP2350_80QFN_minimal: references in all four
  schematics and PCBs to "ProGCC 4 Library"
- Project sym-lib-table and fp-lib-table for all four boards using
  ${KIPRJMOD}-relative paths (replaces Main's absolute fp-lib-table path)

No electrical change. ERC: lib_symbol_issues cleared (Main 70->49,
USBW 36->22, Stick 7->2, Trigger unchanged). DRC unchanged on all boards.

Co-Authored-By: Claude Opus 5.5 <noreply@anthropic.com>
Parts:
- J1, J2: footprint hhl:JST_SM02B-SURS-TF_LF__SN_ -> ProGCC 4 Library:JST_SM02B-SURS-TF_LF__SN_; symbol hhl:SM02B-SURS-TF_LF__SN_ -> ProGCC 4 Library:SM02B-SURS-TF_LF__SN_
- J11, J7: footprint hhl:5051100592 -> ProGCC 4 Library:5051100592
- J3, J5: footprint hhl:5051100892 -> ProGCC 4 Library:5051100892
- J9: footprint hhl:5051101792 -> ProGCC 4 Library:5051101792
- L1: footprint hhl:L_pol_2016 -> ProGCC 4 Library:L_pol_2016
- RGB1, RGB10, RGB11, RGB12, RGB13, RGB14, RGB15, RGB16, RGB2, RGB3, RGB4, RGB5, RGB6, RGB7, RGB8, RGB9: footprint hhl:SK6805-EC-10 -> ProGCC 4 Library:SK6805-EC-10; symbol progcc_v3:SK6805-EC-10 -> ProGCC 4 Library:SK6805-EC-10
- SW10, SW11, SW3, SW4, SW5, SW6, SW7, SW8, SW9: footprint hhl:KSC-TE -> ProGCC 4 Library:KSC-TE
- U1, U10, U11, U3, U6, U7, U8, U9: footprint hhl:SOT-23-5L -> ProGCC 4 Library:SOT-23-5L
- U2: footprint hhl:RP2350-QFN-80-1EP_10x10_P0.4mm_EP3.4x3.4mm_ThermalVias -> ProGCC 4 Library:RP2350-QFN-80-1EP_10x10_P0.4mm_EP3.4x3.4mm_ThermalVias; symbol hhl:RP2350_80QFN -> ProGCC 4 Library:RP2350_80QFN
- U4, U5: footprint hhl:LGA14 -> ProGCC 4 Library:LGA14; symbol progcc_v3:ST_LSM6 -> ProGCC 4 Library:ST_LSM6
Changed lines of the file:
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@@
 			)
 		)
-		(property "Footprint" "hhl:5051100892"
+		(property "Footprint" "ProGCC 4 Library:5051100892"
 			(at 134.62 58.42 0)
 			(hide yes)
@@
 			)
 		)
-		(property "Footprint" "hhl:5051101792"
+		(property "Footprint" "ProGCC 4 Library:5051101792"
 			(at 274.32 93.98 0)
 			(hide yes)
@@
 	)
 	(symbol
-		(lib_id "progcc_v3:SK6805-EC-10")
+		(lib_id "ProGCC 4 Library:SK6805-EC-10")
 		(at 377.19 242.57 0)
 		(unit 1)
@@
 			)
 		)
-		(property "Footprint" "hhl:SK6805-EC-10"
+		(property "Footprint" "ProGCC 4 Library:SK6805-EC-10"
 			(at 377.19 257.81 0)
 			(hide yes)
@@
 	)
 	(symbol
-		(lib_id "progcc_v3:SK6805-EC-10")
+		(lib_id "ProGCC 4 Library:SK6805-EC-10")
 		(at 326.39 242.57 0)
 		(unit 1)
@@
 			)
 		)
-		(property "Footprint" "hhl:SK6805-EC-10"
+		(property "Footprint" "ProGCC 4 Library:SK6805-EC-10"
 			(at 326.39 257.81 0)
 			(hide yes)
@@
 	)
 	(symbol
-		(lib_id "hhl:RP2350_80QFN")
+		(lib_id "ProGCC 4 Library:RP2350_80QFN")
 		(at 105.41 176.53 0)
 		(unit 1)
@@
 			)
 		)
-		(property "Footprint" "hhl:RP2350-QFN-80-1EP_10x10_P0.4mm_EP3.4x3.4mm_ThermalVias"
+		(property "Footprint" "ProGCC 4 Library:RP2350-QFN-80-1EP_10x10_P0.4mm_EP3.4x3.4mm_ThermalVias"
 			(at 86.36 176.53 0)
 			(hide yes)
@@
 	)
 	(symbol
-		(lib_id "progcc_v3:SK6805-EC-10")
+		(lib_id "ProGCC 4 Library:SK6805-EC-10")
 		(at 300.99 185.42 0)
 		(unit 1)
@@
 			)
 		)
-		(property "Footprint" "hhl:SK6805-EC-10"
+		(property "Footprint" "ProGCC 4 Library:SK6805-EC-10"
 			(at 300.99 200.66 0)
 			(hide yes)
@@
 	)
 	(symbol
-		(lib_id "progcc_v3:SK6805-EC-10")
+		(lib_id "ProGCC 4 Library:SK6805-EC-10")
 		(at 300.99 224.79 0)
 		(unit 1)
@@
 			)
 		)
-		(property "Footprint" "hhl:SK6805-EC-10"
+		(property "Footprint" "ProGCC 4 Library:SK6805-EC-10"
 			(at 300.99 240.03 0)
 			(hide yes)
@@
 	)
 	(symbol
-		(lib_id "progcc_v3:ST_LSM6")
+		(lib_id "ProGCC 4 Library:ST_LSM6")
 		(at 218.44 231.14 0)
 		(unit 1)
@@
 			)
 		)
-		(property "Footprint" "hhl:LGA14"
+		(property "Footprint" "ProGCC 4 Library:LGA14"
 			(at 218.44 219.71 0)
 			(hide yes)
@@
 			)
 		)
-		(property "Footprint" "hhl:SOT-23-5L"
+		(property "Footprint" "ProGCC 4 Library:SOT-23-5L"
 			(at 374.65 89.535 0)
 			(hide yes)
@@
 	)
 	(symbol
-		(lib_id "progcc_v3:SK6805-EC-10")
+		(lib_id "ProGCC 4 Library:SK6805-EC-10")
 		(at 351.79 242.57 0)
 		(unit 1)
@@
 			)
 		)
-		(property "Footprint" "hhl:SK6805-EC-10"
+		(property "Footprint" "ProGCC 4 Library:SK6805-EC-10"
 			(at 351.79 257.81 0)
 			(hide yes)
@@
 			)
 		)
-		(property "Footprint" "hhl:5051100592"
+		(property "Footprint" "ProGCC 4 Library:5051100592"
 			(at 248.92 132.08 0)
 			(hide yes)
@@
 			)
 		)
-		(property "Footprint" "hhl:KSC-TE"
+		(property "Footprint" "ProGCC 4 Library:KSC-TE"
 			(at 113.03 49.53 0)
 			(hide yes)
@@
 	)
 	(symbol
-		(lib_id "progcc_v3:SK6805-EC-10")
+		(lib_id "ProGCC 4 Library:SK6805-EC-10")
 		(at 377.19 224.79 0)
 		(unit 1)
@@
 			)
 		)
-		(property "Footprint" "hhl:SK6805-EC-10"
+		(property "Footprint" "ProGCC 4 Library:SK6805-EC-10"
 			(at 377.19 240.03 0)
 			(hide yes)
@@
 			)
 		)
-		(property "Footprint" "hhl:KSC-TE"
+		(property "Footprint" "ProGCC 4 Library:KSC-TE"
 			(at 113.03 27.94 0)
 			(hide yes)
@@
 	)
 	(symbol
-		(lib_id "progcc_v3:SK6805-EC-10")
+		(lib_id "ProGCC 4 Library:SK6805-EC-10")
 		(at 300.99 198.12 0)
 		(unit 1)
@@
 			)
 		)
-		(property "Footprint" "hhl:SK6805-EC-10"
+		(property "Footprint" "ProGCC 4 Library:SK6805-EC-10"
 			(at 300.99 213.36 0)
 			(hide yes)
@@
 			)
 		)
-		(property "Footprint" "hhl:5051100592"
+		(property "Footprint" "ProGCC 4 Library:5051100592"
 			(at 275.59 132.08 0)
 			(hide yes)
@@
 	)
 	(symbol
-		(lib_id "progcc_v3:ST_LSM6")
+		(lib_id "ProGCC 4 Library:ST_LSM6")
 		(at 218.44 191.77 0)
 		(unit 1)
@@
 			)
 		)
-		(property "Footprint" "hhl:LGA14"
+		(property "Footprint" "ProGCC 4 Library:LGA14"
 			(at 218.44 180.34 0)
 			(hide yes)
@@
 	)
 	(symbol
-		(lib_id "progcc_v3:SK6805-EC-10")
+		(lib_id "ProGCC 4 Library:SK6805-EC-10")
 		(at 326.39 185.42 0)
 		(unit 1)
@@
 			)
 		)
-		(property "Footprint" "hhl:SK6805-EC-10"
+		(property "Footprint" "ProGCC 4 Library:SK6805-EC-10"
 			(at 326.39 200.66 0)
 			(hide yes)
@@
 			)
 		)
-		(property "Footprint" "hhl:KSC-TE"
+		(property "Footprint" "ProGCC 4 Library:KSC-TE"
 			(at 113.03 54.61 0)
 			(hide yes)
@@
 			)
 		)
-		(property "Footprint" "hhl:SOT-23-5L"
+		(property "Footprint" "ProGCC 4 Library:SOT-23-5L"
 			(at 328.93 107.315 0)
 			(hide yes)
@@
 	)
 	(symbol
-		(lib_id "hhl:SM02B-SURS-TF_LF__SN_")
+		(lib_id "ProGCC 4 Library:SM02B-SURS-TF_LF__SN_")
 		(at 325.12 31.75 180)
 		(unit 1)
@@
 			)
 		)
-		(property "Footprint" "hhl:JST_SM02B-SURS-TF_LF__SN_"
+		(property "Footprint" "ProGCC 4 Library:JST_SM02B-SURS-TF_LF__SN_"
 			(at 325.12 31.75 0)
 			(hide yes)
@@
 	)
 	(symbol
-		(lib_id "progcc_v3:SK6805-EC-10")
+		(lib_id "ProGCC 4 Library:SK6805-EC-10")
 		(at 351.79 185.42 0)
 		(unit 1)
@@
 			)
 		)
-		(property "Footprint" "hhl:SK6805-EC-10"
+		(property "Footprint" "ProGCC 4 Library:SK6805-EC-10"
 			(at 351.79 200.66 0)
 			(hide yes)
@@
 			)
 		)
-		(property "Footprint" "hhl:SOT-23-5L"
+		(property "Footprint" "ProGCC 4 Library:SOT-23-5L"
 			(at 328.93 125.095 0)
 			(hide yes)
@@
 	)
 	(symbol
-		(lib_id "progcc_v3:SK6805-EC-10")
+		(lib_id "ProGCC 4 Library:SK6805-EC-10")
 		(at 377.19 185.42 0)
 		(unit 1)
@@
 			)
 		)
-		(property "Footprint" "hhl:SK6805-EC-10"
+		(property "Footprint" "ProGCC 4 Library:SK6805-EC-10"
 			(at 377.19 200.66 0)
 			(hide yes)
@@
 	)
 	(symbol
-		(lib_id "hhl:SM02B-SURS-TF_LF__SN_")
+		(lib_id "ProGCC 4 Library:SM02B-SURS-TF_LF__SN_")
 		(at 236.22 31.75 180)
 		(unit 1)
@@
 			)
 		)
-		(property "Footprint" "hhl:JST_SM02B-SURS-TF_LF__SN_"
+		(property "Footprint" "ProGCC 4 Library:JST_SM02B-SURS-TF_LF__SN_"
 			(at 236.22 31.75 0)
 			(hide yes)
@@
 			)
 		)
-		(property "Footprint" "hhl:KSC-TE"
+		(property "Footprint" "ProGCC 4 Library:KSC-TE"
 			(at 113.03 36.83 0)
 			(hide yes)
@@
 			)
 		)
-		(property "Footprint" "hhl:L_pol_2016"
+		(property "Footprint" "ProGCC 4 Library:L_pol_2016"
 			(at 41.91 139.7 0)
 			(hide yes)
@@
 			)
 		)
-		(property "Footprint" "hhl:SOT-23-5L"
+		(property "Footprint" "ProGCC 4 Library:SOT-23-5L"
 			(at 374.65 125.095 0)
 			(hide yes)
@@
 			)
 		)
-		(property "Footprint" "hhl:KSC-TE"
+		(property "Footprint" "ProGCC 4 Library:KSC-TE"
 			(at 113.03 41.91 0)
 			(hide yes)
@@
 			)
 		)
-		(property "Footprint" "hhl:SOT-23-5L"
+		(property "Footprint" "ProGCC 4 Library:SOT-23-5L"
 			(at 328.93 142.875 0)
 			(hide yes)
@@
 			)
 		)
-		(property "Footprint" "hhl:SOT-23-5L"
+		(property "Footprint" "ProGCC 4 Library:SOT-23-5L"
 			(at 374.65 142.875 0)
 			(hide yes)
@@
 	)
 	(symbol
-		(lib_id "progcc_v3:SK6805-EC-10")
+		(lib_id "ProGCC 4 Library:SK6805-EC-10")
 		(at 326.39 224.79 0)
 		(unit 1)
@@
 			)
 		)
-		(property "Footprint" "hhl:SK6805-EC-10"
+		(property "Footprint" "ProGCC 4 Library:SK6805-EC-10"
 			(at 326.39 240.03 0)
 			(hide yes)
@@
 			)
 		)
-		(property "Footprint" "hhl:5051100892"
+		(property "Footprint" "ProGCC 4 Library:5051100892"
 			(at 134.62 33.02 0)
 			(hide yes)
@@
 			)
 		)
-		(property "Footprint" "hhl:KSC-TE"
+		(property "Footprint" "ProGCC 4 Library:KSC-TE"
 			(at 68.58 66.04 0)
 			(hide yes)
@@
 	)
 	(symbol
-		(lib_id "progcc_v3:SK6805-EC-10")
+		(lib_id "ProGCC 4 Library:SK6805-EC-10")
 		(at 351.79 224.79 0)
 		(unit 1)
@@
 			)
 		)
-		(property "Footprint" "hhl:SK6805-EC-10"
+		(property "Footprint" "ProGCC 4 Library:SK6805-EC-10"
 			(at 351.79 240.03 0)
 			(hide yes)
@@
 			)
 		)
-		(property "Footprint" "hhl:KSC-TE"
+		(property "Footprint" "ProGCC 4 Library:KSC-TE"
 			(at 68.58 71.12 0)
 			(hide yes)
@@
 			)
 		)
-		(property "Footprint" "hhl:SOT-23-5L"
+		(property "Footprint" "ProGCC 4 Library:SOT-23-5L"
 			(at 328.93 89.535 0)
 			(hide yes)
@@
 			)
 		)
-		(property "Footprint" "hhl:KSC-TE"
+		(property "Footprint" "ProGCC 4 Library:KSC-TE"
 			(at 113.03 22.86 0)
 			(hide yes)
@@
 			)
 		)
-		(property "Footprint" "hhl:KSC-TE"
+		(property "Footprint" "ProGCC 4 Library:KSC-TE"
 			(at 113.03 63.5 0)
 			(hide yes)
@@
 	)
 	(symbol
-		(lib_id "progcc_v3:SK6805-EC-10")
+		(lib_id "ProGCC 4 Library:SK6805-EC-10")
 		(at 326.39 198.12 0)
 		(unit 1)
@@
 			)
 		)
-		(property "Footprint" "hhl:SK6805-EC-10"
+		(property "Footprint" "ProGCC 4 Library:SK6805-EC-10"
 			(at 326.39 213.36 0)
 			(hide yes)
@@
 	)
 	(symbol
-		(lib_id "progcc_v3:SK6805-EC-10")
+		(lib_id "ProGCC 4 Library:SK6805-EC-10")
 		(at 300.99 242.57 0)
 		(unit 1)
@@
 			)
 		)
-		(property "Footprint" "hhl:SK6805-EC-10"
+		(property "Footprint" "ProGCC 4 Library:SK6805-EC-10"
 			(at 300.99 257.81 0)
 			(hide yes)
@@
 	)
 	(symbol
-		(lib_id "progcc_v3:SK6805-EC-10")
+		(lib_id "ProGCC 4 Library:SK6805-EC-10")
 		(at 377.19 198.12 0)
 		(unit 1)
@@
 			)
 		)
-		(property "Footprint" "hhl:SK6805-EC-10"
+		(property "Footprint" "ProGCC 4 Library:SK6805-EC-10"
 			(at 377.19 213.36 0)
 			(hide yes)
@@
 	)
 	(symbol
-		(lib_id "progcc_v3:SK6805-EC-10")
+		(lib_id "ProGCC 4 Library:SK6805-EC-10")
 		(at 351.79 198.12 0)
 		(unit 1)
@@
 			)
 		)
-		(property "Footprint" "hhl:SK6805-EC-10"
+		(property "Footprint" "ProGCC 4 Library:SK6805-EC-10"
 			(at 351.79 213.36 0)
 			(hide yes)
@@
 			)
 		)
-		(property "Footprint" "hhl:SOT-23-5L"
+		(property "Footprint" "ProGCC 4 Library:SOT-23-5L"
 			(at 374.65 107.315 0)
 			(hide yes)

Commit message: Add HAL4395 symbol and swap it in for the hall sensors
New ProGCC 4 Library:HAL4395 (1 VCC, 2 ~EN, 3 GND, 4 NC, 5 OUT tri-state),
geometry identical to the patched placeholder so no wiring changes.
Replaces Regulator_Linear:TLV70012_SOT23-5 on the 8 Main and 4 Trigger FPC
halls. Clears the hall lib_symbol_mismatch warnings and the shared-ADC
output-to-output pin conflicts. Netlist unchanged (checked against kicad-cli).

Co-Authored-By: Claude Opus 5.5 <noreply@anthropic.com>
Parts:
- U1, U10, U11, U3, U6, U7, U8, U9: symbol Regulator_Linear:TLV70012_SOT23-5 -> ProGCC 4 Library:HAL4395
Changed lines of the file:
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@@
 	)
 	(symbol
-		(lib_id "Regulator_Linear:TLV70012_SOT23-5")
+		(lib_id "ProGCC 4 Library:HAL4395")
 		(at 374.65 97.79 0)
 		(unit 1)
@@
 			)
 		)
-		(property "Description" "SOT-23-5L Linear, Compass (ICs) ROHS"
+		(property "Description" "Linear Hall-effect sensor, ratiometric analog output, active-low enable, tri-state output when disabled, SOT-23-5L"
 			(at 377.698 92.71 0)
 			(hide yes)
@@
 	)
 	(symbol
-		(lib_id "Regulator_Linear:TLV70012_SOT23-5")
+		(lib_id "ProGCC 4 Library:HAL4395")
 		(at 328.93 115.57 0)
 		(unit 1)
@@
 			)
 		)
-		(property "Description" "SOT-23-5L Linear, Compass (ICs) ROHS"
+		(property "Description" "Linear Hall-effect sensor, ratiometric analog output, active-low enable, tri-state output when disabled, SOT-23-5L"
 			(at 331.978 110.49 0)
 			(hide yes)
@@
 	)
 	(symbol
-		(lib_id "Regulator_Linear:TLV70012_SOT23-5")
+		(lib_id "ProGCC 4 Library:HAL4395")
 		(at 328.93 133.35 0)
 		(unit 1)
@@
 			)
 		)
-		(property "Description" "SOT-23-5L Linear, Compass (ICs) ROHS"
+		(property "Description" "Linear Hall-effect sensor, ratiometric analog output, active-low enable, tri-state output when disabled, SOT-23-5L"
 			(at 331.978 128.27 0)
 			(hide yes)
@@
 	)
 	(symbol
-		(lib_id "Regulator_Linear:TLV70012_SOT23-5")
+		(lib_id "ProGCC 4 Library:HAL4395")
 		(at 374.65 133.35 0)
 		(unit 1)
@@
 			)
 		)
-		(property "Description" "SOT-23-5L Linear, Compass (ICs) ROHS"
+		(property "Description" "Linear Hall-effect sensor, ratiometric analog output, active-low enable, tri-state output when disabled, SOT-23-5L"
 			(at 377.698 128.27 0)
 			(hide yes)
@@
 	)
 	(symbol
-		(lib_id "Regulator_Linear:TLV70012_SOT23-5")
+		(lib_id "ProGCC 4 Library:HAL4395")
 		(at 328.93 151.13 0)
 		(unit 1)
@@
 			)
 		)
-		(property "Description" "SOT-23-5L Linear, Compass (ICs) ROHS"
+		(property "Description" "Linear Hall-effect sensor, ratiometric analog output, active-low enable, tri-state output when disabled, SOT-23-5L"
 			(at 331.978 146.05 0)
 			(hide yes)
@@
 	)
 	(symbol
-		(lib_id "Regulator_Linear:TLV70012_SOT23-5")
+		(lib_id "ProGCC 4 Library:HAL4395")
 		(at 374.65 151.13 0)
 		(unit 1)
@@
 			)
 		)
-		(property "Description" "SOT-23-5L Linear, Compass (ICs) ROHS"
+		(property "Description" "Linear Hall-effect sensor, ratiometric analog output, active-low enable, tri-state output when disabled, SOT-23-5L"
 			(at 377.698 146.05 0)
 			(hide yes)
@@
 	)
 	(symbol
-		(lib_id "Regulator_Linear:TLV70012_SOT23-5")
+		(lib_id "ProGCC 4 Library:HAL4395")
 		(at 328.93 97.79 0)
 		(unit 1)
@@
 			)
 		)
-		(property "Description" "SOT-23-5L Linear, Compass (ICs) ROHS"
+		(property "Description" "Linear Hall-effect sensor, ratiometric analog output, active-low enable, tri-state output when disabled, SOT-23-5L"
 			(at 331.978 92.71 0)
 			(hide yes)
@@
 	)
 	(symbol
-		(lib_id "Regulator_Linear:TLV70012_SOT23-5")
+		(lib_id "ProGCC 4 Library:HAL4395")
 		(at 374.65 115.57 0)
 		(unit 1)
@@
 			)
 		)
-		(property "Description" "SOT-23-5L Linear, Compass (ICs) ROHS"
+		(property "Description" "Linear Hall-effect sensor, ratiometric analog output, active-low enable, tri-state output when disabled, SOT-23-5L"
 			(at 377.698 110.49 0)
 			(hide yes)

Commit message: Main: ERC cleanup and PWR_FLAGs
- No-connect flags on unused RP2354B pins (GPIO22-27, GPIO36-39, QSPI
  SD0-3/SCLK; flash is internal) and on RGB2/4/6/8 DOUT (paired LEDs).
- Remove the dangling wire stubs on GPIO36-38.
- PWR_FLAGs on GND, +3V3 (from J9), +1V1 (VREG via L1) and VREG_AVDD
  (via R11).
- ST_LSM6: VDD/VDDIO/GND/GNDIO retyped bidirectional -> power_in.
- Refresh embedded MMBT2222A from the KiCad 10 library (pins unchanged).

ERC 37 -> 13. Netlist unchanged (checked against kicad-cli).

Co-Authored-By: Claude Opus 5.5 <noreply@anthropic.com>
Connections:
- no-connect marks 8 -> 27

Commit message: BOM fields: fill missing MPN/LCSC, drop empty legacy fields
- Main: MPN/LCSC for R1/R28/R29 (1k), R5/R6 (10k), R7/R8 (100R),
  R11 (33R, RC0201FR-0733RL / C295794) and R9/R10 (10R). R9/R10's Link
  pointed at the 0R jumper (C106227); corrected to RC0201FR-0710RL /
  C106226 to match the 10R value.
- USBW: R38 Manufacturer YAGEO; trim trailing whitespace on 9 MPNs.
- Trigger FPC: J1/J2 are the ribbon-tail fingers, not purchased parts;
  exclude from BOM and position files.
- All boards: remove properties with empty values (Manufacturer_Name,
  Mouser fields, Height, JLCPN, PART_REV, etc.). Populated fields and
  the standard/core fields are untouched.

SW1 (GuliKit stick) and P1 (RM2) have no LCSC number by design.
ERC counts and netlists unchanged.

Co-Authored-By: Claude Opus 5.5 <noreply@anthropic.com>
Parts:
- R1, R28, R29: LCSC (none) -> C138165; MPN (none) -> RC0201FR-071KL
- R10, R9: LCSC (none) -> C106226; Link https://www.lcsc.com/product-detail/Chip-Resistor-Surface-M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 -> https://www.lcsc.com/product-detail/C106226.html; MPN (none) -> RC0201FR-0710RL
- R11: LCSC (none) -> C295794; MPN (none) -> RC0201FR-0733RL
- R5, R6: LCSC (none) -> C106225; MPN (none) -> RC0201FR-0710KL
- R7, R8: LCSC (none) -> C77623; MPN (none) -> RC0201FR-07100RL
