File: PCB/Projects/Trigger FPC/FPC_Trigger_Board.kicad_pcb (KiCad board)
At the start: 2 copper layers, 74.6 x 20.7 mm, 10 parts, among them J1 Conn_01x05_Pin, J2 Conn_01x05_Pin, U1 HAL4395, U2 HAL4395, U3 HAL4395, U4 HAL4395

Commit message: Consolidate custom symbols, footprints and 3D models into repo library
Make the hardware repo self-contained instead of depending on the external
HHL-KiCad-Lib checkout and the missing progcc_v3 symbol library.

- New PCB/Libraries/ProGCC 4 Library.kicad_sym: the 12 custom symbols,
  extracted from the schematics' embedded caches (identical to what the
  boards use; duplicate hhl/progcc_v3 CUS08F30 merged)
- Library.pretty: add the 7 missing footprints and replace 9 that differed
  from the placed footprints with the hhl copies the boards match
- PCB/Libraries/3dmodels: STEP models previously referenced by absolute
  path into HHL-KiCad-Lib, now via ${KIPRJMOD}/../../Libraries/3dmodels
- Relink hhl:/progcc_v3:/RP2350_80QFN_minimal: references in all four
  schematics and PCBs to "ProGCC 4 Library"
- Project sym-lib-table and fp-lib-table for all four boards using
  ${KIPRJMOD}-relative paths (replaces Main's absolute fp-lib-table path)

No electrical change. ERC: lib_symbol_issues cleared (Main 70->49,
USBW 36->22, Stick 7->2, Trigger unchanged). DRC unchanged on all boards.

Co-Authored-By: Claude Opus 5.5 <noreply@anthropic.com>
Parts:
- J1, J2: footprint hhl:505110-0592 Ribbon -> ProGCC 4 Library:505110-0592 Ribbon
- U1, U2, U3, U4: footprint hhl:SOT-23-5L -> ProGCC 4 Library:SOT-23-5L
Changed lines of the file:
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@@
 		)
 	)
-	(footprint "hhl:SOT-23-5L"
+	(footprint "ProGCC 4 Library:SOT-23-5L"
 		(layer "F.Cu")
 		(at 241.408396 156.966586 -90)
@@
 		)
 	)
-	(footprint "hhl:SOT-23-5L"
+	(footprint "ProGCC 4 Library:SOT-23-5L"
 		(layer "F.Cu")
 		(at 230.213014 156.966586 -90)
@@
 		)
 	)
-	(footprint "hhl:SOT-23-5L"
+	(footprint "ProGCC 4 Library:SOT-23-5L"
 		(layer "F.Cu")
 		(at 230.213144 144.905691 -90)
@@
 		)
 	)
-	(footprint "hhl:SOT-23-5L"
+	(footprint "ProGCC 4 Library:SOT-23-5L"
 		(layer "F.Cu")
 		(at 241.408267 144.905691 -90)
@@
 		)
 	)
-	(footprint "hhl:505110-0592 Ribbon"
+	(footprint "ProGCC 4 Library:505110-0592 Ribbon"
 		(layer "B.Cu")
 		(at 199.95 160.6 -90)
@@
 		(embedded_fonts no)
 	)
-	(footprint "hhl:505110-0592 Ribbon"
+	(footprint "ProGCC 4 Library:505110-0592 Ribbon"
 		(layer "B.Cu")
 		(at 271.575 160.6 -90)
