File: PCB/Projects/Trigger FPC/FPC_Trigger_Board.kicad_pcb (KiCad board)
At the start: 2 copper layers, 74.6 x 20.7 mm, 10 parts, among them J1 Conn_01x05_Pin, J2 Conn_01x05_Pin, U1 HAL4395, U2 HAL4395, U3 HAL4395, U4 HAL4395

Commit message: Trigger FPC: ground the back pours with stitching vias, refill zones
Add 2 GND and 2 GNDL vias (0.6/0.3) in the sensor areas so the hatched
B.Cu pours are tied to ground instead of floating. Zones refilled.

DRC: 0 errors, isolated-copper warnings cleared. Remaining warnings
are cosmetic: 0201 lib mismatch (4), silk clipped (2), text height (8).

Co-Authored-By: Claude Opus 5.5 <noreply@anthropic.com>
Routing:
- net GNDL: vias 0 -> 2
- net GND: vias 0 -> 2
Changed lines of the file:
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@@
 		(capping no)
 		(filling no)
+		(zone_defaults)
 		(pcbplotparams
 			(layerselection 0x00000000_00000000_555555d5_5755fdff)
@@
 		(net "GNDL")
 	)
+	(via
+		(at 240.125 152.675)
+		(size 0.6)
+		(drill 0.3)
+		(layers "F.Cu" "B.Cu")
+		(free yes)
+		(net "GNDL")
+	)
+	(via
+		(at 240.2 151.4)
+		(size 0.6)
+		(drill 0.3)
+		(layers "F.Cu" "B.Cu")
+		(free yes)
+		(net "GNDL")
+	)
 	(segment
 		(start 271.075001 154.850001)
@@
 		(net "GND")
 	)
+	(via
+		(at 232.35 149.65)
+		(size 0.6)
+		(drill 0.3)
+		(layers "F.Cu" "B.Cu")
+		(free yes)
+		(net "GND")
+	)
+	(via
+		(at 232.375 150.875)
+		(size 0.6)
+		(drill 0.3)
+		(layers "F.Cu" "B.Cu")
+		(free yes)
+		(net "GND")
+	)
 	(segment
 		(start 228.525 159.9)
@@
 	)
 	(segment
+		(start 241.408 145.133)
+		(end 241.408 146.6)
+		(width 0.2)
+		(layer "F.Cu")
+		(net "ADC_2")
+	)
+	(segment
 		(start 242.925 153.55)
 		(end 270.475 153.55)
@@
 	)
 	(segment
-		(start 241.408 145.133)
-		(end 241.408 146.6)
+		(start 241.8 152.425)
+		(end 242.925 153.55)
 		(width 0.2)
 		(layer "F.Cu")
@@
 		(width 0.2)
 		(layer "F.Cu")
-		(net "ADC_2")
-	)
-	(segment
-		(start 241.8 152.425)
-		(end 242.925 153.55)
-		(width 0.2)
-		(layer "F.Cu")
