File: PCB/Projects/Trigger FPC/FPC_Trigger_Board.kicad_sch (KiCad schematic)
At the start: 10 parts, among them J1 Conn_01x05_Pin, J2 Conn_01x05_Pin, U1 HAL4395, U2 HAL4395, U3 HAL4395, U4 HAL4395

Commit message: Consolidate custom symbols, footprints and 3D models into repo library
Make the hardware repo self-contained instead of depending on the external
HHL-KiCad-Lib checkout and the missing progcc_v3 symbol library.

- New PCB/Libraries/ProGCC 4 Library.kicad_sym: the 12 custom symbols,
  extracted from the schematics' embedded caches (identical to what the
  boards use; duplicate hhl/progcc_v3 CUS08F30 merged)
- Library.pretty: add the 7 missing footprints and replace 9 that differed
  from the placed footprints with the hhl copies the boards match
- PCB/Libraries/3dmodels: STEP models previously referenced by absolute
  path into HHL-KiCad-Lib, now via ${KIPRJMOD}/../../Libraries/3dmodels
- Relink hhl:/progcc_v3:/RP2350_80QFN_minimal: references in all four
  schematics and PCBs to "ProGCC 4 Library"
- Project sym-lib-table and fp-lib-table for all four boards using
  ${KIPRJMOD}-relative paths (replaces Main's absolute fp-lib-table path)

No electrical change. ERC: lib_symbol_issues cleared (Main 70->49,
USBW 36->22, Stick 7->2, Trigger unchanged). DRC unchanged on all boards.

Co-Authored-By: Claude Opus 5.5 <noreply@anthropic.com>
Parts:
- J1, J2: footprint hhl:505110-0592 Ribbon -> ProGCC 4 Library:505110-0592 Ribbon
- U1, U2, U3, U4: footprint hhl:SOT-23-5L -> ProGCC 4 Library:SOT-23-5L
Changed lines of the file:
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@@
 			)
 		)
-		(property "Footprint" "hhl:505110-0592 Ribbon"
+		(property "Footprint" "ProGCC 4 Library:505110-0592 Ribbon"
 			(at 21.59 127 0)
 			(hide yes)
@@
 			)
 		)
-		(property "Footprint" "hhl:505110-0592 Ribbon"
+		(property "Footprint" "ProGCC 4 Library:505110-0592 Ribbon"
 			(at 21.59 107.95 0)
 			(hide yes)
@@
 			)
 		)
-		(property "Footprint" "hhl:SOT-23-5L"
+		(property "Footprint" "ProGCC 4 Library:SOT-23-5L"
 			(at 35.56 50.165 0)
 			(hide yes)
@@
 			)
 		)
-		(property "Footprint" "hhl:SOT-23-5L"
+		(property "Footprint" "ProGCC 4 Library:SOT-23-5L"
 			(at 114.3 50.165 0)
 			(hide yes)
@@
 			)
 		)
-		(property "Footprint" "hhl:SOT-23-5L"
+		(property "Footprint" "ProGCC 4 Library:SOT-23-5L"
 			(at 74.93 50.165 0)
 			(hide yes)
@@
 			)
 		)
-		(property "Footprint" "hhl:SOT-23-5L"
+		(property "Footprint" "ProGCC 4 Library:SOT-23-5L"
 			(at 153.67 50.165 0)
 			(hide yes)

Commit message: Add HAL4395 symbol and swap it in for the hall sensors
New ProGCC 4 Library:HAL4395 (1 VCC, 2 ~EN, 3 GND, 4 NC, 5 OUT tri-state),
geometry identical to the patched placeholder so no wiring changes.
Replaces Regulator_Linear:TLV70012_SOT23-5 on the 8 Main and 4 Trigger FPC
halls. Clears the hall lib_symbol_mismatch warnings and the shared-ADC
output-to-output pin conflicts. Netlist unchanged (checked against kicad-cli).

Co-Authored-By: Claude Opus 5.5 <noreply@anthropic.com>
Parts:
- U1, U2, U3, U4: symbol Regulator_Linear:TLV70012_SOT23-5 -> ProGCC 4 Library:HAL4395
Changed lines of the file:
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@@
 	)
 	(symbol
-		(lib_id "Regulator_Linear:TLV70012_SOT23-5")
+		(lib_id "ProGCC 4 Library:HAL4395")
 		(at 35.56 58.42 0)
 		(unit 1)
@@
 			)
 		)
-		(property "Description" "SOT-23-5L Linear, Compass (ICs) ROHS"
+		(property "Description" "Linear Hall-effect sensor, ratiometric analog output, active-low enable, tri-state output when disabled, SOT-23-5L"
 			(at 38.608 53.34 0)
 			(hide yes)
@@
 	)
 	(symbol
-		(lib_id "Regulator_Linear:TLV70012_SOT23-5")
+		(lib_id "ProGCC 4 Library:HAL4395")
 		(at 114.3 58.42 0)
 		(unit 1)
@@
 			)
 		)
-		(property "Description" "SOT-23-5L Linear, Compass (ICs) ROHS"
+		(property "Description" "Linear Hall-effect sensor, ratiometric analog output, active-low enable, tri-state output when disabled, SOT-23-5L"
 			(at 117.348 53.34 0)
 			(hide yes)
@@
 	)
 	(symbol
-		(lib_id "Regulator_Linear:TLV70012_SOT23-5")
+		(lib_id "ProGCC 4 Library:HAL4395")
 		(at 74.93 58.42 0)
 		(unit 1)
@@
 			)
 		)
-		(property "Description" "SOT-23-5L Linear, Compass (ICs) ROHS"
+		(property "Description" "Linear Hall-effect sensor, ratiometric analog output, active-low enable, tri-state output when disabled, SOT-23-5L"
 			(at 77.978 53.34 0)
 			(hide yes)
@@
 	)
 	(symbol
-		(lib_id "Regulator_Linear:TLV70012_SOT23-5")
+		(lib_id "ProGCC 4 Library:HAL4395")
 		(at 153.67 58.42 0)
 		(unit 1)
@@
 			)
 		)
-		(property "Description" "SOT-23-5L Linear, Compass (ICs) ROHS"
+		(property "Description" "Linear Hall-effect sensor, ratiometric analog output, active-low enable, tri-state output when disabled, SOT-23-5L"
 			(at 156.718 53.34 0)
 			(hide yes)

Commit message: BOM fields: fill missing MPN/LCSC, drop empty legacy fields
- Main: MPN/LCSC for R1/R28/R29 (1k), R5/R6 (10k), R7/R8 (100R),
  R11 (33R, RC0201FR-0733RL / C295794) and R9/R10 (10R). R9/R10's Link
  pointed at the 0R jumper (C106227); corrected to RC0201FR-0710RL /
  C106226 to match the 10R value.
- USBW: R38 Manufacturer YAGEO; trim trailing whitespace on 9 MPNs.
- Trigger FPC: J1/J2 are the ribbon-tail fingers, not purchased parts;
  exclude from BOM and position files.
- All boards: remove properties with empty values (Manufacturer_Name,
  Mouser fields, Height, JLCPN, PART_REV, etc.). Populated fields and
  the standard/core fields are untouched.

SW1 (GuliKit stick) and P1 (RM2) have no LCSC number by design.
ERC counts and netlists unchanged.

Co-Authored-By: Claude Opus 5.5 <noreply@anthropic.com>
Parts:
- J1, J2: now left out of the parts list
