File: PCB/Projects/Stick Board/PGS_Stick_Board.kicad_pcb (KiCad board)
At the start: 2 copper layers, 37.5 x 29.7 mm, 10 parts, among them J1 Molex 505110-0892, SW1 GL1807SYAE-002

Commit message: Sync local board work; replace Trigger Board with Trigger FPC
- Update Main, Stick and USBW board layouts, schematics and 3D exports
- Replace the rigid Trigger Board project with the new Trigger FPC design
- Add shared PCB/Libraries footprint library and fp-lib-table
- Regenerate production outputs (gerbers, drills, placement, BOM) for all boards
- Stop tracking KiCad auto-backup folders and fp-info-cache; consolidate .gitignore

Co-Authored-By: Claude Opus 5 <noreply@anthropic.com>
Parts:
- C1, C2: footprint Capacitor_SMD:C_0603_1608Metric -> Capacitor_SMD:C_0402_1005Metric
- moved C1 0.70 mm to (63.1, 48.6)
- moved C2 0.64 mm to (51.0, 60.4)
Routing:
- net RGB_OUT: track 18.6 -> 16.5 mm
- net OUT_X: track 41.5 -> 40.8 mm
Other:
- board text added: "PGC 4.0 Stick Module"
- board text removed: "ProGCC 4 Stick Module"

Commit message: Consolidate custom symbols, footprints and 3D models into repo library
Make the hardware repo self-contained instead of depending on the external
HHL-KiCad-Lib checkout and the missing progcc_v3 symbol library.

- New PCB/Libraries/ProGCC 4 Library.kicad_sym: the 12 custom symbols,
  extracted from the schematics' embedded caches (identical to what the
  boards use; duplicate hhl/progcc_v3 CUS08F30 merged)
- Library.pretty: add the 7 missing footprints and replace 9 that differed
  from the placed footprints with the hhl copies the boards match
- PCB/Libraries/3dmodels: STEP models previously referenced by absolute
  path into HHL-KiCad-Lib, now via ${KIPRJMOD}/../../Libraries/3dmodels
- Relink hhl:/progcc_v3:/RP2350_80QFN_minimal: references in all four
  schematics and PCBs to "ProGCC 4 Library"
- Project sym-lib-table and fp-lib-table for all four boards using
  ${KIPRJMOD}-relative paths (replaces Main's absolute fp-lib-table path)

No electrical change. ERC: lib_symbol_issues cleared (Main 70->49,
USBW 36->22, Stick 7->2, Trigger unchanged). DRC unchanged on all boards.

Co-Authored-By: Claude Opus 5.5 <noreply@anthropic.com>
Parts:
- J1: footprint hhl:5051100892 -> ProGCC 4 Library:5051100892
- RGB1, RGB2, RGB3, RGB4: footprint hhl:SK6805-EC-10 -> ProGCC 4 Library:SK6805-EC-10
- SW1: footprint hhl:GL1807SYAE -> ProGCC 4 Library:GL1807SYAE
Changed lines of the file:
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@@
 		)
 	)
-	(footprint "hhl:SK6805-EC-10"
+	(footprint "ProGCC 4 Library:SK6805-EC-10"
 		(layer "F.Cu")
 		(at 59.725 54.955329)
@@
 		)
 	)
-	(footprint "hhl:SK6805-EC-10"
+	(footprint "ProGCC 4 Library:SK6805-EC-10"
 		(layer "F.Cu")
 		(at 42.725 41.955329)
@@
 		)
 	)
-	(footprint "hhl:SK6805-EC-10"
+	(footprint "ProGCC 4 Library:SK6805-EC-10"
 		(layer "F.Cu")
 		(at 59.725 41.955329)
@@
 		)
 	)
-	(footprint "hhl:5051100892"
+	(footprint "ProGCC 4 Library:5051100892"
 		(layer "F.Cu")
 		(at 33.65 36.35 180)
@@
 		)
 	)
-	(footprint "hhl:SK6805-EC-10"
+	(footprint "ProGCC 4 Library:SK6805-EC-10"
 		(layer "F.Cu")
 		(at 42.725 54.955329)
@@
 		)
 	)
-	(footprint "hhl:GL1807SYAE"
+	(footprint "ProGCC 4 Library:GL1807SYAE"
 		(layer "F.Cu")
 		(at 51.225 48.455329)
