File: PCB/Projects/Stick Board/PGS_Stick_Board.kicad_pcb (KiCad board)
At the start: 2 copper layers, 37.5 x 29.7 mm, 10 parts, among them J1 Molex 505110-0892, SW1 GL1807SYAE-002

Commit message: Stick PCB: fix DRC errors (short, outline, dangling via, clearance)
- Delete an orphan OUT_Y track stub between C1's pads that shorted
  OUT_Y to GND (also the solder-mask bridge). OUT_Y still reaches C1
  pad 2 via its existing track.
- Delete a 17 nm Edge.Cuts segment and close the 17 nm gap by moving
  the adjoining line's endpoint (malformed outline).
- Delete the dangling +3V3 via at (59.225, 56.525); its two F.Cu tracks
  already meet there.
- Default net class clearance 0.2 -> 0.15 mm so the stock 0201
  footprints (0.18 mm pad gap) pass; Main uses 0.1 mm.

DRC 22 -> 16 (with zone refill). Remaining: J1 MP2 tab edge clearance
(accepted), J1 silk clipped by edge, R1/R2 library mismatch, text height.

Co-Authored-By: Claude Opus 5.5 <noreply@anthropic.com>
Routing:
- net +3V3: vias 6 -> 5
Changed lines of the file:
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@@
 	(gr_line
 		(start 37.082864 60.476144)
-		(end 39.204173 62.597454)
+		(end 39.204185 62.597442)
 		(stroke
 			(width 0.01)
@@
 		(start 38.302495 55.720979)
 		(end 37.082865 56.940609)
-		(stroke
-			(width 0.01)
-			(type default)
-		)
-		(layer "Edge.Cuts")
-	)
-	(gr_line
-		(start 39.204185 62.597442)
-		(end 39.204173 62.597454)
 		(stroke
 			(width 0.01)
@@
 	)
 	(via
-		(at 59.225 56.525)
-		(size 0.6)
-		(drill 0.3)
-		(layers "F.Cu" "B.Cu")
-		(capping no)
-		(covering
-			(front no)
-			(back no)
-		)
-		(plugging
-			(front no)
-			(back no)
-		)
-		(filling no)
-		(net "+3V3")
-	)
-	(via
 		(at 55.325 58.225)
 		(size 0.6)
@@
 		(width 0.2)
 		(layer "F.Cu")
-		(net "OUT_Y")
-	)
-	(segment
-		(start 62.9 48.775329)
-		(end 62.9 48.480329)
-		(width 0.2)
-		(layer "F.Cu")
