File: PCB/Projects/Stick Board/PGS_Stick_Board.kicad_sch (KiCad schematic)
At the start: 10 parts, among them J1 Molex 505110-0892, SW1 GL1807SYAE-002

Commit message: Sync local board work; replace Trigger Board with Trigger FPC
- Update Main, Stick and USBW board layouts, schematics and 3D exports
- Replace the rigid Trigger Board project with the new Trigger FPC design
- Add shared PCB/Libraries footprint library and fp-lib-table
- Regenerate production outputs (gerbers, drills, placement, BOM) for all boards
- Stop tracking KiCad auto-backup folders and fp-info-cache; consolidate .gitignore

Co-Authored-By: Claude Opus 5 <noreply@anthropic.com>
Parts:
- C1, C2: footprint Capacitor_SMD:C_0603_1608Metric -> Capacitor_SMD:C_0402_1005Metric; LCSC C519554 -> C272875; MPN CC0603JRX7R9BB473 -> CC0402KRX7R9BB473
Other:
- company: Hand Held Legend, LLC -> Hand Held Legend LLC
- title: ProGCC 4 Stick Module -> PGC Joystick Module

Commit message: Consolidate custom symbols, footprints and 3D models into repo library
Make the hardware repo self-contained instead of depending on the external
HHL-KiCad-Lib checkout and the missing progcc_v3 symbol library.

- New PCB/Libraries/ProGCC 4 Library.kicad_sym: the 12 custom symbols,
  extracted from the schematics' embedded caches (identical to what the
  boards use; duplicate hhl/progcc_v3 CUS08F30 merged)
- Library.pretty: add the 7 missing footprints and replace 9 that differed
  from the placed footprints with the hhl copies the boards match
- PCB/Libraries/3dmodels: STEP models previously referenced by absolute
  path into HHL-KiCad-Lib, now via ${KIPRJMOD}/../../Libraries/3dmodels
- Relink hhl:/progcc_v3:/RP2350_80QFN_minimal: references in all four
  schematics and PCBs to "ProGCC 4 Library"
- Project sym-lib-table and fp-lib-table for all four boards using
  ${KIPRJMOD}-relative paths (replaces Main's absolute fp-lib-table path)

No electrical change. ERC: lib_symbol_issues cleared (Main 70->49,
USBW 36->22, Stick 7->2, Trigger unchanged). DRC unchanged on all boards.

Co-Authored-By: Claude Opus 5.5 <noreply@anthropic.com>
Parts:
- J1: footprint hhl:5051100892 -> ProGCC 4 Library:5051100892
- RGB1, RGB2, RGB3, RGB4: footprint hhl:SK6805-EC-10 -> ProGCC 4 Library:SK6805-EC-10; symbol progcc_v3:SK6805-EC-10 -> ProGCC 4 Library:SK6805-EC-10
- SW1: footprint hhl:GL1807SYAE -> ProGCC 4 Library:GL1807SYAE; symbol progcc_v3:GL1807SYAE-002 -> ProGCC 4 Library:GL1807SYAE-002
Changed lines of the file:
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@@
 			)
 		)
-		(property "Footprint" "hhl:5051100892"
+		(property "Footprint" "ProGCC 4 Library:5051100892"
 			(at 86.36 24.13 0)
 			(hide yes)
@@
 	)
 	(symbol
-		(lib_id "progcc_v3:SK6805-EC-10")
+		(lib_id "ProGCC 4 Library:SK6805-EC-10")
 		(at 110.49 58.42 0)
 		(unit 1)
@@
 			)
 		)
-		(property "Footprint" "hhl:SK6805-EC-10"
+		(property "Footprint" "ProGCC 4 Library:SK6805-EC-10"
 			(at 110.49 73.66 0)
 			(hide yes)
@@
 	)
 	(symbol
-		(lib_id "progcc_v3:SK6805-EC-10")
+		(lib_id "ProGCC 4 Library:SK6805-EC-10")
 		(at 59.69 58.42 0)
 		(unit 1)
@@
 			)
 		)
-		(property "Footprint" "hhl:SK6805-EC-10"
+		(property "Footprint" "ProGCC 4 Library:SK6805-EC-10"
 			(at 59.69 73.66 0)
 			(hide yes)
@@
 	)
 	(symbol
-		(lib_id "progcc_v3:SK6805-EC-10")
+		(lib_id "ProGCC 4 Library:SK6805-EC-10")
 		(at 85.09 58.42 0)
 		(unit 1)
@@
 			)
 		)
-		(property "Footprint" "hhl:SK6805-EC-10"
+		(property "Footprint" "ProGCC 4 Library:SK6805-EC-10"
 			(at 85.09 73.66 0)
 			(hide yes)
@@
 	)
 	(symbol
-		(lib_id "progcc_v3:GL1807SYAE-002")
+		(lib_id "ProGCC 4 Library:GL1807SYAE-002")
 		(at 54.61 22.86 0)
 		(unit 1)
@@
 			)
 		)
-		(property "Footprint" "hhl:GL1807SYAE"
+		(property "Footprint" "ProGCC 4 Library:GL1807SYAE"
 			(at 55.88 34.798 0)
 			(hide yes)
@@
 	)
 	(symbol
-		(lib_id "progcc_v3:SK6805-EC-10")
+		(lib_id "ProGCC 4 Library:SK6805-EC-10")
 		(at 34.29 58.42 0)
 		(unit 1)
@@
 			)
 		)
-		(property "Footprint" "hhl:SK6805-EC-10"
+		(property "Footprint" "ProGCC 4 Library:SK6805-EC-10"
 			(at 34.29 73.66 0)
 			(hide yes)

Commit message: Stick: correct C1/C2 package and description
MPN CC0402KRX7R9BB473 / LCSC C272875 is YAGEO 0402, 47nF, ±10%, 50V,
X7R (LCSC listing; K = ±10%, 9 = 50V in YAGEO CC ordering codes), which
matches the 0402 footprint. The Package field said 0603 and the
descriptions said 0603 (C1 also ±5%); now "0402" and
"CAP CER 47nF 50V X7R ±10% 0402".

Co-Authored-By: Claude Opus 5.5 <noreply@anthropic.com>
Parts:
- C1, C2: Package 0603 -> 0402
Changed lines of the file:
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@@
 			)
 		)
-		(property "Description" "CAP CER 47nF 50V X7R 0603"
+		(property "Description" "CAP CER 47nF 50V X7R ±10% 0402"
 			(at 34.29 35.56 0)
 			(hide yes)
@@
 			)
 		)
-		(property "Package" "0603"
+		(property "Package" "0402"
 			(at 34.29 35.56 0)
 			(hide yes)
@@
 			)
 		)
-		(property "Description" "50V 47nF X7R ±5% 0603"
+		(property "Description" "CAP CER 47nF 50V X7R ±10% 0402"
 			(at 22.86 34.29 0)
 			(hide yes)
@@
 			)
 		)
-		(property "Package" "0603"
+		(property "Package" "0402"
 			(at 22.86 34.29 0)
 			(hide yes)
