File: PCB/Projects/USBW Board/PGS_USBW_Board.kicad_sch (KiCad schematic)
At the start: 47 parts, among them IC1 BQ27621YZFR-G1A, J1 Molex 505110-1792, J2 USB4056-03-A, J4 PH 2.0 JST, P1 RPI-RM2, Q1 BSS138DW, Q2 BSS138DW, U1 USBLC6-2P6, U2 USBLC6-2P6, U3 USBLC6-2P6, U4 TPS63001DRCR, U5 BQ25180

Commit message: Sync local board work; replace Trigger Board with Trigger FPC
- Update Main, Stick and USBW board layouts, schematics and 3D exports
- Replace the rigid Trigger Board project with the new Trigger FPC design
- Add shared PCB/Libraries footprint library and fp-lib-table
- Regenerate production outputs (gerbers, drills, placement, BOM) for all boards
- Stop tracking KiCad auto-backup folders and fp-info-cache; consolidate .gitignore

Co-Authored-By: Claude Opus 5 <noreply@anthropic.com>
Parts:
- added R38: 100k, Resistor_SMD:R_0402_1005Metric, symbol Device:R_Small
Connections:
- net +3.3V_PRE: now also R38.1
- net GND: now also R38.2
Other:
- company: (none) -> Hand Held Legend LLC
- title: (none) -> PGC USB+W Module

Commit message: Consolidate custom symbols, footprints and 3D models into repo library
Make the hardware repo self-contained instead of depending on the external
HHL-KiCad-Lib checkout and the missing progcc_v3 symbol library.

- New PCB/Libraries/ProGCC 4 Library.kicad_sym: the 12 custom symbols,
  extracted from the schematics' embedded caches (identical to what the
  boards use; duplicate hhl/progcc_v3 CUS08F30 merged)
- Library.pretty: add the 7 missing footprints and replace 9 that differed
  from the placed footprints with the hhl copies the boards match
- PCB/Libraries/3dmodels: STEP models previously referenced by absolute
  path into HHL-KiCad-Lib, now via ${KIPRJMOD}/../../Libraries/3dmodels
- Relink hhl:/progcc_v3:/RP2350_80QFN_minimal: references in all four
  schematics and PCBs to "ProGCC 4 Library"
- Project sym-lib-table and fp-lib-table for all four boards using
  ${KIPRJMOD}-relative paths (replaces Main's absolute fp-lib-table path)

No electrical change. ERC: lib_symbol_issues cleared (Main 70->49,
USBW 36->22, Stick 7->2, Trigger unchanged). DRC unchanged on all boards.

Co-Authored-By: Claude Opus 5.5 <noreply@anthropic.com>
Parts:
- D1, D3: symbol progcc_v3:CUS08F30 -> ProGCC 4 Library:CUS08F30
- D4: symbol hhl:CUS08F30 -> ProGCC 4 Library:CUS08F30
- IC1: footprint hhl:BGA9C50P3X3_162X158X62 -> ProGCC 4 Library:BGA9C50P3X3_162X158X62; symbol hhl:BQ27621YZFR-G1A -> ProGCC 4 Library:BQ27621YZFR-G1A
- J1: footprint hhl:5051101792 -> ProGCC 4 Library:5051101792
- J2: footprint hhl:USB405603A -> ProGCC 4 Library:USB405603A; symbol hhl:USB4056-03-A -> ProGCC 4 Library:USB4056-03-A
- P1: footprint hhl:RPI_RM2 -> ProGCC 4 Library:RPI_RM2; symbol hhl:RPI-RM2 -> ProGCC 4 Library:RPI-RM2
- Q1, Q2: symbol hhl:BSS138DW -> ProGCC 4 Library:BSS138DW
- U4: footprint hhl:VREG_V62_16624-01YE -> ProGCC 4 Library:VREG_V62_16624-01YE; symbol hhl:TPS63000DRCR -> ProGCC 4 Library:TPS63000DRCR
- U5: footprint hhl:DSBGA -> ProGCC 4 Library:DSBGA; symbol hhl:BQ25180 -> ProGCC 4 Library:BQ25180
Changed lines of the file:
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@@
 	)
 	(symbol
-		(lib_id "progcc_v3:CUS08F30")
+		(lib_id "ProGCC 4 Library:CUS08F30")
 		(at 138.43 44.45 90)
 		(unit 1)
@@
 	)
 	(symbol
-		(lib_id "progcc_v3:CUS08F30")
+		(lib_id "ProGCC 4 Library:CUS08F30")
 		(at 212.09 22.86 270)
 		(unit 1)
@@
 	)
 	(symbol
-		(lib_id "hhl:RPI-RM2")
+		(lib_id "ProGCC 4 Library:RPI-RM2")
 		(at 109.22 172.72 0)
 		(unit 2)
@@
 			)
 		)
-		(property "Footprint" "hhl:RPI_RM2"
+		(property "Footprint" "ProGCC 4 Library:RPI_RM2"
 			(at 109.474 156.972 0)
 			(hide yes)
@@
 	)
 	(symbol
-		(lib_id "hhl:BSS138DW")
+		(lib_id "ProGCC 4 Library:BSS138DW")
 		(at 236.22 27.94 0)
 		(mirror y)
@@
 	)
 	(symbol
-		(lib_id "hhl:CUS08F30")
+		(lib_id "ProGCC 4 Library:CUS08F30")
 		(at 114.3 118.11 180)
 		(unit 1)
@@
 			)
 		)
-		(property "Footprint" "hhl:5051101792"
+		(property "Footprint" "ProGCC 4 Library:5051101792"
 			(at 176.53 139.7 0)
 			(hide yes)
@@
 	)
 	(symbol
-		(lib_id "hhl:BSS138DW")
+		(lib_id "ProGCC 4 Library:BSS138DW")
 		(at 257.81 67.31 0)
 		(mirror y)
@@
 	)
 	(symbol
-		(lib_id "hhl:BSS138DW")
+		(lib_id "ProGCC 4 Library:BSS138DW")
 		(at 257.81 38.1 0)
 		(mirror y)
@@
 	)
 	(symbol
-		(lib_id "hhl:USB4056-03-A")
+		(lib_id "ProGCC 4 Library:USB4056-03-A")
 		(at 228.6 121.92 0)
 		(unit 1)
@@
 			)
 		)
-		(property "Footprint" "hhl:USB405603A"
+		(property "Footprint" "ProGCC 4 Library:USB405603A"
 			(at 257.81 216.84 0)
 			(hide yes)
@@
 	)
 	(symbol
-		(lib_id "hhl:BQ27621YZFR-G1A")
+		(lib_id "ProGCC 4 Library:BQ27621YZFR-G1A")
 		(at 45.72 105.41 0)
 		(unit 1)
@@
 			)
 		)
-		(property "Footprint" "hhl:BGA9C50P3X3_162X158X62"
+		(property "Footprint" "ProGCC 4 Library:BGA9C50P3X3_162X158X62"
 			(at 72.39 200.33 0)
 			(hide yes)
@@
 	)
 	(symbol
-		(lib_id "hhl:BSS138DW")
+		(lib_id "ProGCC 4 Library:BSS138DW")
 		(at 257.81 96.52 0)
 		(mirror y)
@@
 	)
 	(symbol
-		(lib_id "hhl:RPI-RM2")
+		(lib_id "ProGCC 4 Library:RPI-RM2")
 		(at 143.51 172.72 0)
 		(unit 3)
@@
 			)
 		)
-		(property "Footprint" "hhl:RPI_RM2"
+		(property "Footprint" "ProGCC 4 Library:RPI_RM2"
 			(at 143.764 156.972 0)
 			(hide yes)
@@
 	)
 	(symbol
-		(lib_id "hhl:TPS63000DRCR")
+		(lib_id "ProGCC 4 Library:TPS63000DRCR")
 		(at 191.77 43.18 0)
 		(unit 1)
@@
 			)
 		)
-		(property "Footprint" "hhl:VREG_V62_16624-01YE"
+		(property "Footprint" "ProGCC 4 Library:VREG_V62_16624-01YE"
 			(at 191.77 43.18 0)
 			(hide yes)
@@
 	)
 	(symbol
-		(lib_id "hhl:BQ25180")
+		(lib_id "ProGCC 4 Library:BQ25180")
 		(at 120.65 100.33 0)
 		(unit 1)
@@
 			)
 		)
-		(property "Footprint" "hhl:DSBGA"
+		(property "Footprint" "ProGCC 4 Library:DSBGA"
 			(at 120.65 100.33 0)
 			(hide yes)
@@
 	)
 	(symbol
-		(lib_id "hhl:RPI-RM2")
+		(lib_id "ProGCC 4 Library:RPI-RM2")
 		(at 143.51 144.78 0)
 		(unit 1)
@@
 			)
 		)
-		(property "Footprint" "hhl:RPI_RM2"
+		(property "Footprint" "ProGCC 4 Library:RPI_RM2"
 			(at 143.764 129.032 0)
 			(hide yes)
