File: PCB/Projects/USBW Board/PGS_USBW_Board.kicad_sch (KiCad schematic)
At the start: 48 parts, among them IC1 BQ27621YZFR-G1A, J1 Molex 505110-1792, J2 USB4056-03-A, J4 PH 2.0 JST, P1 RPI-RM2, Q1 BSS138DW, Q2 BSS138DW, U1 USBLC6-2P6, U2 USBLC6-2P6, U3 USBLC6-2P6, U4 TPS63001DRCR, U5 BQ25180

Commit message: BOM fields: fill missing MPN/LCSC, drop empty legacy fields
- Main: MPN/LCSC for R1/R28/R29 (1k), R5/R6 (10k), R7/R8 (100R),
  R11 (33R, RC0201FR-0733RL / C295794) and R9/R10 (10R). R9/R10's Link
  pointed at the 0R jumper (C106227); corrected to RC0201FR-0710RL /
  C106226 to match the 10R value.
- USBW: R38 Manufacturer YAGEO; trim trailing whitespace on 9 MPNs.
- Trigger FPC: J1/J2 are the ribbon-tail fingers, not purchased parts;
  exclude from BOM and position files.
- All boards: remove properties with empty values (Manufacturer_Name,
  Mouser fields, Height, JLCPN, PART_REV, etc.). Populated fields and
  the standard/core fields are untouched.

SW1 (GuliKit stick) and P1 (RM2) have no LCSC number by design.
ERC counts and netlists unchanged.

Co-Authored-By: Claude Opus 5.5 <noreply@anthropic.com>
Parts:
- D1, D3, D4: MPN CUS08F30,H3F -> CUS08F30,H3F
- R10: MPN RC0201FR-070RL -> RC0201FR-070RL
- R12, R13, R20, R29: MPN RC0201FR-0710KL -> RC0201FR-0710KL
- R38: Manufacturer (none) -> YAGEO
- R9: MPN RC0201FR-07100RL -> RC0201FR-07100RL

Commit message: USBW: fix TPS63000 EP pins and test-point position-file flags
- TPS63000DRCR: remove stacked pins 11_1..11_8 (library + embedded +
  U4 instance). The VREG_V62_16624-01YE footprint has a single custom
  EP pad "11", so these caused "pad not found" errors on PCB update.
  They sat on pin 11, so connectivity is unchanged (EP still on GND).
- TP1-TP7: in_pos_files no, matching the PCB. Otherwise the update
  would strip the PCB's position-file exclusion.

ERC unchanged (5). Netlist matches kicad-cli.

Co-Authored-By: Claude Opus 5.5 <noreply@anthropic.com>
Connections:
- net GND: no longer U4.11_1 (EP), U4.11_2 (EP), U4.11_3 (EP), U4.11_4 (EP), U4.11_5 (EP), U4.11_6 (EP), U4.11_7 (EP), U4.11_8 (EP)
Changed lines of the file:
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@@
 		(in_bom no)
 		(on_board yes)
-		(in_pos_files yes)
+		(in_pos_files no)
 		(dnp yes)
 		(property "Reference" "TP5"
@@
 		(in_bom no)
 		(on_board yes)
-		(in_pos_files yes)
+		(in_pos_files no)
 		(dnp yes)
 		(property "Reference" "TP2"
@@
 		(in_bom no)
 		(on_board yes)
-		(in_pos_files yes)
+		(in_pos_files no)
 		(dnp yes)
 		(property "Reference" "TP4"
@@
 		(in_bom no)
 		(on_board yes)
-		(in_pos_files yes)
+		(in_pos_files no)
 		(dnp yes)
 		(property "Reference" "TP6"
@@
 		(in_bom no)
 		(on_board yes)
-		(in_pos_files yes)
+		(in_pos_files no)
 		(dnp yes)
 		(property "Reference" "TP3"
@@
 		(in_bom no)
 		(on_board yes)
-		(in_pos_files yes)
+		(in_pos_files no)
 		(dnp yes)
 		(property "Reference" "TP1"
@@
 		(pin "11"
 		)
-		(pin "11_1"
-		)
-		(pin "11_2"
-		)
-		(pin "11_3"
-		)
-		(pin "11_4"
-		)
-		(pin "11_5"
-		)
-		(pin "11_6"
-		)
-		(pin "11_7"
-		)
-		(pin "11_8"
-		)
 		(pin "2"
 		)
@@
 		(in_bom no)
 		(on_board yes)
-		(in_pos_files yes)
+		(in_pos_files no)
 		(dnp yes)
 		(property "Reference" "TP7"
